File: Hardware/SWAFarmNodeV1/SWAFarmNodeV1.kicad_pcb (KiCad board)
At the start: 2 copper layers, 0 parts

Commit message: updated
Parts:
- added C_BST1: 0.1uF, Capacitor_SMD:C_0603_1608Metric, F.Cu at (1.50, 24.4)
- added C_FF1: 10pF, Capacitor_SMD:C_0603_1608Metric, F.Cu at (1.50, 26.9)
- added C_INTVCC1: 2.2uF, Capacitor_SMD:C_0805_2012Metric, F.Cu at (26.3, 28.6)
- added C_SS1: 10nF, Capacitor_SMD:C_0603_1608Metric, F.Cu at (1.50, 29.4)
- added Cin1: 10uF_50V, Capacitor_SMD:C_1210_3225Metric, F.Cu at (22.4, 15.1)
- added Cin2: 10uF_50V, Capacitor_SMD:C_1210_3225Metric, F.Cu at (22.4, 19.4)
- added Cout1: 22uF_16V, Capacitor_SMD:C_1206_3216Metric, F.Cu at (28.1, 14.7)
- added Cout2: 22uF_16V, Capacitor_SMD:C_1206_3216Metric, F.Cu at (28.1, 18.0)
- added D1: SMBJ16CA, Diode_SMD:D_SMB, F.Cu at (23.8, 24.3)
- added D_LED1: LED_Green_2mA, LED_SMD:LED_0805_2012Metric, F.Cu at (21.9, 28.6)
- added F1: 1.1A_Hold_PTC, Fuse:Fuse_1812_4532Metric, F.Cu at (7.38, 29.3)
- added J1: DC_IN_12V, TerminalBlock_Phoenix:TerminalBlock_Phoenix_MKDS-3-2-5.08_1x02_P5.08mm_Horizontal, F.Cu at (7.47, 6.42)
- added L1: 4.7uH, Inductor_SMD:L_10.4x10.4_H4.8, F.Cu at (22.4, 5.47)
- added Q1: NMOS_30V_RDSon_20mOhm, Package_TO_SOT_SMD:TO-252-2, F.Cu at (10.8, 17.2)
- added R1: 24.0k_1%, Resistor_SMD:R_0805_2012Metric, F.Cu at (1.71, 0.97)
- added R2: 10.0k_1%, Resistor_SMD:R_0805_2012Metric, F.Cu at (1.71, 3.92)
- added R_EN_BOT1: 100k, Resistor_SMD:R_0805_2012Metric, F.Cu at (1.71, 6.88)
- added R_EN_TOP1: 787k, Resistor_SMD:R_0805_2012Metric, F.Cu at (1.71, 9.82)
- added R_LED1: 680, Resistor_SMD:R_0805_2012Metric, F.Cu at (1.71, 12.8)
- added R_PG1: 100k, Resistor_SMD:R_0805_2012Metric, F.Cu at (1.71, 15.7)
- added R_RT1: 41.2k, Resistor_SMD:R_0805_2012Metric, F.Cu at (1.71, 18.7)
- added R_gate1: 10k, Resistor_SMD:R_0805_2012Metric, F.Cu at (1.71, 21.6)
- added TP1: VIN_PROT, TestPoint:TestPoint_THTPad_1.5x1.5mm_Drill0.7mm, F.Cu at (17.8, 14.8)
- added TP2: 3V3_RAIL, TestPoint:TestPoint_THTPad_1.5x1.5mm_Drill0.7mm, F.Cu at (17.8, 18.3)
- added TP3: GND, TestPoint:TestPoint_THTPad_1.5x1.5mm_Drill0.7mm, F.Cu at (17.8, 21.9)
- added TP4: PG, TestPoint:TestPoint_THTPad_1.5x1.5mm_Drill0.7mm, F.Cu at (17.8, 25.4)
- added U1: LT8610AC-3.3, Package_SO:MSOP-16-1EP_3x4.039mm_P0.5mm_EP1.651x2.845mm_ThermalVias, F.Cu at (7.94, 24.0)

Commit message: updated upto  step 9 - PCB Floor Planning & Component Placement
Parts:
- added C_BATSENSE1: 100nF, C_0603_1608Metric, F.Cu at (177.0, 78.0)
- added C_BTN1: 100nF, C_0603_1608Metric, F.Cu at (251.0, 145.0)
- added C_BTST1: 100nF, C_0603_1608Metric, F.Cu at (30.0, 66.0)
- added C_BTST2: 100nF, C_0603_1608Metric, F.Cu at (30.0, 72.0)
- added C_CAP1_1: 1uF, C_0805_2012Metric, F.Cu at (185.0, 44.0)
- added C_LORA_VDD1: 100nF, C_0603_1608Metric, F.Cu at (215.0, 20.0)
- added C_LSE1: 8pF, C_0603_1608Metric, F.Cu at (178.0, 124.0)
- added C_LSE2: 8pF, C_0603_1608Metric, F.Cu at (184.0, 124.0)
- added C_MCU_BULK1: 4.7uF, C_0805_2012Metric, F.Cu at (167.0, 100.0)
- added C_MCU_VBAT1: 100nF, C_0603_1608Metric, F.Cu at (125.0, 100.0)
- added C_MCU_VDD1: 100nF, C_0603_1608Metric, F.Cu at (131.0, 100.0)
- added C_MCU_VDD2: 100nF, C_0603_1608Metric, F.Cu at (137.0, 100.0)
- added C_MCU_VDD3: 100nF, C_0603_1608Metric, F.Cu at (143.0, 100.0)
- added C_MCU_VDDA1: 1uF, C_0603_1608Metric, F.Cu at (149.0, 100.0)
- added C_MCU_VDDA2: 100nF, C_0603_1608Metric, F.Cu at (155.0, 100.0)
- added C_MCU_VDDUSB1: 100nF, C_0603_1608Metric, F.Cu at (161.0, 100.0)
- added C_NRST1: 100nF, C_0603_1608Metric, F.Cu at (115.0, 138.0)
- added C_PMID1: 10uF, C_1210_3225Metric, F.Cu at (75.0, 60.0)
- added C_REGN1: 1uF, C_0805_2012Metric, F.Cu at (75.0, 66.0)
- added C_REGOUT1: 1uF, C_0805_2012Metric, F.Cu at (185.0, 50.0)
- added C_RELAY_BULK1: 22uF, C_1210_3225Metric, F.Cu at (100.0, 202.0)
- added C_RS485_VCC1: 100nF, C_0603_1608Metric, F.Cu at (68.0, 126.0)
- added C_SOL_IN1: 4.7uF, C_0805_2012Metric, F.Cu at (70.0, 44.0)
- added C_SYS1: 22uF, C_1210_3225Metric, F.Cu at (90.0, 60.0)
- added C_VC1_1: 100nF, C_0603_1608Metric, F.Cu at (191.0, 60.0)
- added C_VC2_1: 100nF, C_0603_1608Metric, F.Cu at (191.0, 66.0)
- added C_VC3_1: 100nF, C_0603_1608Metric, F.Cu at (191.0, 72.0)
- added D2: SMBJ24A_class_unidirectional, D_SMB, F.Cu at (55.0, 44.0)
- added D_ACT1: LED_Yellow_activity, LED_0805_2012Metric, F.Cu at (220.0, 145.0)
- added D_CHG_STAT1: LED_Yellow_charge_status, LED_0805_2012Metric, F.Cu at (30.0, 84.0)
- added D_RELAY1_FLYBACK1: S1M_1A_1000V_SMA, D_SMA, F.Cu at (130.0, 172.0)
- added D_RELAY1_STATUS1: LED_Green_relay_status, LED_0805_2012Metric, F.Cu at (106.0, 164.0)
- added D_RELAY2_FLYBACK1: S1M_1A_1000V_SMA, D_SMA, F.Cu at (167.0, 172.0)
- added D_RELAY2_STATUS1: LED_Green_relay_status, LED_0805_2012Metric, F.Cu at (143.0, 164.0)
- added D_RELAY3_FLYBACK1: S1M_1A_1000V_SMA, D_SMA, F.Cu at (204.0, 172.0)
- added D_RELAY3_STATUS1: LED_Green_relay_status, LED_0805_2012Metric, F.Cu at (180.0, 164.0)
- added D_RELAY4_FLYBACK1: S1M_1A_1000V_SMA, D_SMA, F.Cu at (241.0, 172.0)
- added D_RELAY4_STATUS1: LED_Green_relay_status, LED_0805_2012Metric, F.Cu at (217.0, 164.0)
- added D_RELAY5_FLYBACK1: S1M_1A_1000V_SMA, D_SMA, F.Cu at (278.0, 172.0)
- added D_RELAY5_STATUS1: LED_Green_relay_status, LED_0805_2012Metric, F.Cu at (254.0, 164.0)
- added D_RS485_TVS_A1: SMBJ_class_RS485, D_SMB, F.Cu at (68.0, 92.0)
- added D_RS485_TVS_B1: SMBJ_class_RS485, D_SMB, F.Cu at (76.0, 92.0)
- added D_SENSOR_PWR_TVS1: SMBJ18A_class_unidirectional, D_SMB, F.Cu at (84.0, 92.0)
- added D_STATUS1: LED_Green_status, LED_0805_2012Metric, F.Cu at (178.0, 135.0)
- added F2: 0.75A_Hold_PTC, Fuse_1812_4532Metric, F.Cu at (55.0, 32.0)
- added F3: 10A_series_onetime, Fuse_1206_3216Metric, F.Cu at (150.0, 32.0)
- added FB_MCU1: BLM18 class, L_0603_1608Metric, F.Cu at (173.0, 100.0)
- added FB_RELAY_PWR1: Power Ferrite, 1A class, L_1206_3216Metric, F.Cu at (100.0, 196.0)
- added F_RS485_A1: 0.2A_Hold_PTC, Fuse_1206_3216Metric, F.Cu at (45.0, 94.0)
- added F_RS485_A2: 0.2A_Hold_PTC, Fuse_1206_3216Metric, F.Cu at (45.0, 118.0)
- added F_RS485_A3: 0.2A_Hold_PTC, Fuse_1206_3216Metric, F.Cu at (45.0, 142.0)
- added F_RS485_A4: 0.2A_Hold_PTC, Fuse_1206_3216Metric, F.Cu at (45.0, 166.0)
- added F_RS485_A5: 0.2A_Hold_PTC, Fuse_1206_3216Metric, F.Cu at (45.0, 190.0)
- added F_RS485_B1: 0.2A_Hold_PTC, Fuse_1206_3216Metric, F.Cu at (45.0, 102.0)
- added F_RS485_B2: 0.2A_Hold_PTC, Fuse_1206_3216Metric, F.Cu at (45.0, 126.0)
- added F_RS485_B3: 0.2A_Hold_PTC, Fuse_1206_3216Metric, F.Cu at (45.0, 150.0)
- added F_RS485_B4: 0.2A_Hold_PTC, Fuse_1206_3216Metric, F.Cu at (45.0, 174.0)
- added F_RS485_B5: 0.2A_Hold_PTC, Fuse_1206_3216Metric, F.Cu at (45.0, 198.0)
- added F_RS485_PWR1: 0.2A_Hold_PTC, Fuse_1206_3216Metric, F.Cu at (55.0, 98.0)
- added F_RS485_PWR2: 0.2A_Hold_PTC, Fuse_1206_3216Metric, F.Cu at (55.0, 122.0)
- added F_RS485_PWR3: 0.2A_Hold_PTC, Fuse_1206_3216Metric, F.Cu at (55.0, 146.0)
- added F_RS485_PWR4: 0.2A_Hold_PTC, Fuse_1206_3216Metric, F.Cu at (55.0, 170.0)
- added F_RS485_PWR5: 0.2A_Hold_PTC, Fuse_1206_3216Metric, F.Cu at (55.0, 194.0)
- added J2: SOLAR_IN_12V_class, TerminalBlock_Phoenix_MKDS-3-2-5.08_1x02_P5.08mm_Horizontal, F.Cu at (55.0, 18.0)
- added J3: 4S_LiFePO4_Pack, TerminalBlock_Phoenix_MKDS-3-2-5.08_1x02_P5.08mm_Horizontal, F.Cu at (150.0, 18.0)
- added J_DBG_UART1: Debug_Console, PinHeader_1x03_P2.54mm_Vertical, F.Cu at (240.0, 122.0)
- added J_LORA_ANT1: U.FL_to_SMA_pigtail, U.FL_Hirose_U.FL-R-SMT-1_Vertical, F.Cu at (275.0, 22.0)
- added J_RELAY11: Relay1_COM_NO_NC, TerminalBlock_Phoenix_MKDS-1,5-3-5.08_1x03_P5.08mm_Horizontal, F.Cu at (118.0, 208.0)
- added J_RELAY21: Relay2_COM_NO_NC, TerminalBlock_Phoenix_MKDS-1,5-3-5.08_1x03_P5.08mm_Horizontal, F.Cu at (155.0, 208.0)
- added J_RELAY31: Relay3_COM_NO_NC, TerminalBlock_Phoenix_MKDS-1,5-3-5.08_1x03_P5.08mm_Horizontal, F.Cu at (192.0, 208.0)
- added J_RELAY41: Relay4_COM_NO_NC, TerminalBlock_Phoenix_MKDS-1,5-3-5.08_1x03_P5.08mm_Horizontal, F.Cu at (229.0, 208.0)
- added J_RELAY51: Relay5_COM_NO_NC, TerminalBlock_Phoenix_MKDS-1,5-3-5.08_1x03_P5.08mm_Horizontal, F.Cu at (266.0, 208.0)
- added J_RS485_SENSOR1: Sensor1_A_B_PWR_GND, TerminalBlock_Phoenix_MKDS-1,5-4-5.08_1x04_P5.08mm_Horizontal, F.Cu at (22.0, 98.0)
- added J_RS485_SENSOR2: Sensor2_A_B_PWR_GND, TerminalBlock_Phoenix_MKDS-1,5-4-5.08_1x04_P5.08mm_Horizontal, F.Cu at (22.0, 122.0)
- added J_RS485_SENSOR3: Sensor3_A_B_PWR_GND, TerminalBlock_Phoenix_MKDS-1,5-4-5.08_1x04_P5.08mm_Horizontal, F.Cu at (22.0, 146.0)
- added J_RS485_SENSOR4: Sensor4_A_B_PWR_GND, TerminalBlock_Phoenix_MKDS-1,5-4-5.08_1x04_P5.08mm_Horizontal, F.Cu at (22.0, 170.0)
- added J_RS485_SENSOR5: Sensor5_A_B_PWR_GND, TerminalBlock_Phoenix_MKDS-1,5-4-5.08_1x04_P5.08mm_Horizontal, F.Cu at (22.0, 194.0)
- added J_SWD1: SWD_ARM10, PinHeader_2x05_P1.27mm_Vertical, F.Cu at (240.0, 105.0)
- added K_RELAY11: FINDER-40.51.9.012.0000_12VDC_SPDT_10A, Relay_SPDT_Finder_40.51, F.Cu at (118.0, 188.0)
- added K_RELAY21: FINDER-40.51.9.012.0000_12VDC_SPDT_10A, Relay_SPDT_Finder_40.51, F.Cu at (155.0, 188.0)
- added K_RELAY31: FINDER-40.51.9.012.0000_12VDC_SPDT_10A, Relay_SPDT_Finder_40.51, F.Cu at (192.0, 188.0)
- added K_RELAY41: FINDER-40.51.9.012.0000_12VDC_SPDT_10A, Relay_SPDT_Finder_40.51, F.Cu at (229.0, 188.0)
- added K_RELAY51: FINDER-40.51.9.012.0000_12VDC_SPDT_10A, Relay_SPDT_Finder_40.51, F.Cu at (266.0, 188.0)
- added L_CHG1: 2.2uH_5A_class, L_10.4x10.4_H4.8, F.Cu at (92.0, 68.0)
- added MH1: MountingHole_3.2mm_M3, MountingHole_3.2mm_M3, F.Cu at (10.0, 10.0)
- added MH2: MountingHole_3.2mm_M3, MountingHole_3.2mm_M3, F.Cu at (293.0, 10.0)
- added MH3: MountingHole_3.2mm_M3, MountingHole_3.2mm_M3, F.Cu at (10.0, 213.0)
- added MH4: MountingHole_3.2mm_M3, MountingHole_3.2mm_M3, F.Cu at (293.0, 213.0)
- added NTC_CHG1: 10k_NTC_-20to60C_class, R_0805_2012Metric, F.Cu at (62.0, 84.0)
- added NTC_PROT1: 10k_NTC_-20to60C_class, R_0805_2012Metric, F.Cu at (185.0, 80.0)
- added Q2: NMOS_30V_RDSon_20mOhm, TO-252-2, F.Cu at (55.0, 56.0)
- added Q_AC1: NMOS_30V_RDSon_20mOhm, TO-252-2, F.Cu at (14.0, 72.0)
- added Q_AC2: NMOS_30V_RDSon_20mOhm, TO-252-2, F.Cu at (14.0, 88.0)
- added Q_CHG1: NMOS_30V_RDSon_20mOhm, TO-252-2, F.Cu at (145.0, 78.0)
- added Q_DSG1: NMOS_30V_RDSon_20mOhm, TO-252-2, F.Cu at (145.0, 66.0)
- added Q_RELAY11: NMOS_30V_RDSon_100mOhm_SOT23, SOT-23, F.Cu at (106.0, 172.0)
- added Q_RELAY21: NMOS_30V_RDSon_100mOhm_SOT23, SOT-23, F.Cu at (143.0, 172.0)
- added Q_RELAY31: NMOS_30V_RDSon_100mOhm_SOT23, SOT-23, F.Cu at (180.0, 172.0)
- added Q_RELAY41: NMOS_30V_RDSon_100mOhm_SOT23, SOT-23, F.Cu at (217.0, 172.0)
- added Q_RELAY51: NMOS_30V_RDSon_100mOhm_SOT23, SOT-23, F.Cu at (254.0, 172.0)
- added R_ACT1: 1k, R_0805_2012Metric, F.Cu at (226.0, 145.0)
- added R_BATSENSE_BOT1: 180k, R_0805_2012Metric, F.Cu at (171.0, 78.0)
- added R_BATSENSE_TOP1: 680k, R_0805_2012Metric, F.Cu at (165.0, 78.0)
- added R_BIAS_PD1: 560, R_0805_2012Metric, F.Cu at (68.0, 118.0)
- added R_BIAS_PU1: 560, R_0805_2012Metric, F.Cu at (74.0, 118.0)
- added R_BOOT0_1: 10k, R_0805_2012Metric, F.Cu at (115.0, 118.0)
- added R_BTN1: 10k, R_0805_2012Metric, F.Cu at (245.0, 145.0)
- added R_CHG_STAT1: 1k, R_0805_2012Metric, F.Cu at (36.0, 84.0)
- added R_I2C_SCL_PU1: 4.7k, R_0805_2012Metric, F.Cu at (105.0, 50.0)
- added R_I2C_SDA_PU1: 4.7k, R_0805_2012Metric, F.Cu at (100.0, 50.0)
- added R_ILIM1: TBD_verify_datasheet_ILIM_formula, R_0805_2012Metric, F.Cu at (75.0, 72.0)
- added R_LORA_BOOT1: 10k, R_0805_2012Metric, F.Cu at (215.0, 36.0)
- added R_LORA_RST1: 10k, R_0805_2012Metric, F.Cu at (215.0, 28.0)
- added R_NRST1: 10k, R_0805_2012Metric, F.Cu at (115.0, 132.0)
- added R_PROG1: TBD_verify_datasheet_for_1.6A_target, R_0805_2012Metric, F.Cu at (75.0, 78.0)
- added R_QON1: 100k, R_0805_2012Metric, F.Cu at (22.0, 88.0)
- added R_RELAY1_GATE1: 100, R_0603_1608Metric, F.Cu at (114.0, 168.0)
- added R_RELAY1_PD1: 10k, R_0603_1608Metric, F.Cu at (122.0, 168.0)
- added R_RELAY1_STATUS1: 1k, R_0805_2012Metric, F.Cu at (130.0, 164.0)
- added R_RELAY2_GATE1: 100, R_0603_1608Metric, F.Cu at (151.0, 168.0)
- added R_RELAY2_PD1: 10k, R_0603_1608Metric, F.Cu at (159.0, 168.0)
- added R_RELAY2_STATUS1: 1k, R_0805_2012Metric, F.Cu at (167.0, 164.0)
- added R_RELAY3_GATE1: 100, R_0603_1608Metric, F.Cu at (188.0, 168.0)
- added R_RELAY3_PD1: 10k, R_0603_1608Metric, F.Cu at (196.0, 168.0)
- added R_RELAY3_STATUS1: 1k, R_0805_2012Metric, F.Cu at (204.0, 164.0)
- added R_RELAY4_GATE1: 100, R_0603_1608Metric, F.Cu at (225.0, 168.0)
- added R_RELAY4_PD1: 10k, R_0603_1608Metric, F.Cu at (233.0, 168.0)
- added R_RELAY4_STATUS1: 1k, R_0805_2012Metric, F.Cu at (241.0, 164.0)
- added R_RELAY5_GATE1: 100, R_0603_1608Metric, F.Cu at (262.0, 168.0)
- added R_RELAY5_PD1: 10k, R_0603_1608Metric, F.Cu at (270.0, 168.0)
- added R_RELAY5_STATUS1: 1k, R_0805_2012Metric, F.Cu at (278.0, 164.0)
- added R_SENSE1: 5mOhm_1percent_2512, R_2512_6332Metric, F.Cu at (145.0, 88.0)
- added R_STATUS1: 330, R_0805_2012Metric, F.Cu at (184.0, 135.0)
- added R_TERM1: 120, R_0805_2012Metric, F.Cu at (80.0, 118.0)
- added R_VC1_1: 1k, R_0603_1608Metric, F.Cu at (185.0, 60.0)
- added R_VC2_1: 1k, R_0603_1608Metric, F.Cu at (185.0, 66.0)
- added R_VC3_1: 1k, R_0603_1608Metric, F.Cu at (185.0, 72.0)
- added R_gate2: 10k, R_0805_2012Metric, F.Cu at (63.0, 56.0)
- added SW_DIP1: TERM_BIAS_SELECT, SW_DIP_SPSTx03_Slide_9.78x9.8mm_W7.62mm_P2.54mm, F.Cu at (92.0, 105.0)
- added SW_RESET1: Reset_Button, SW_SPST_TL3342, F.Cu at (268.0, 150.0)
- added SW_USER1: User_Button, SW_SPST_TL3342, F.Cu at (235.0, 150.0)
- added TP_BAT1: BAT_P, TestPoint_THTPad_1.5x1.5mm_Drill0.7mm, F.Cu at (62.0, 46.0)
- added TP_BATSENSE1: BATSENSE_MID, TestPoint_THTPad_1.5x1.5mm_Drill0.7mm, F.Cu at (165.0, 84.0)
- added TP_BOOT0_1: BOOT0, TestPoint_THTPad_1.5x1.5mm_Drill0.7mm, F.Cu at (115.0, 124.0)
- added TP_ISENSE_HI1: SRP, TestPoint_THTPad_1.5x1.5mm_Drill0.7mm, F.Cu at (152.0, 88.0)
- added TP_ISENSE_LO1: SRN_GND, TestPoint_THTPad_1.5x1.5mm_Drill0.7mm, F.Cu at (158.0, 88.0)
- added TP_LORA_BOOT1: LORA_BOOT0, TestPoint_THTPad_1.5x1.5mm_Drill0.7mm, F.Cu at (271.0, 75.0)
- added TP_LORA_RESET1: LORA_RESET_N, TestPoint_THTPad_1.5x1.5mm_Drill0.7mm, F.Cu at (265.0, 75.0)
- added TP_LORA_RX1: LORA_RX, TestPoint_THTPad_1.5x1.5mm_Drill0.7mm, F.Cu at (265.0, 85.0)
- added TP_LORA_STATUS1: LORA_STATUS, TestPoint_THTPad_1.5x1.5mm_Drill0.7mm, F.Cu at (265.0, 80.0)
- added TP_LORA_SWCLK1: LORA_SWCLK, TestPoint_THTPad_1.5x1.5mm_Drill0.7mm, F.Cu at (265.0, 90.0)
- added TP_LORA_SWDIO1: LORA_SWDIO, TestPoint_THTPad_1.5x1.5mm_Drill0.7mm, F.Cu at (271.0, 85.0)
- added TP_LORA_TX1: LORA_TX, TestPoint_THTPad_1.5x1.5mm_Drill0.7mm, F.Cu at (271.0, 80.0)
- added TP_MCU_RX1: MCU_RX, TestPoint_THTPad_1.5x1.5mm_Drill0.7mm, F.Cu at (226.0, 122.0)
- added TP_MCU_TX1: MCU_TX, TestPoint_THTPad_1.5x1.5mm_Drill0.7mm, F.Cu at (220.0, 122.0)
- added TP_NRST1: NRST, TestPoint_THTPad_1.5x1.5mm_Drill0.7mm, F.Cu at (121.0, 138.0)
- added TP_RELAY1_CTRL1: RELAY1_CTRL, TestPoint_THTPad_1.5x1.5mm_Drill0.7mm, F.Cu at (118.0, 160.0)
- added TP_RELAY2_CTRL1: RELAY2_CTRL, TestPoint_THTPad_1.5x1.5mm_Drill0.7mm, F.Cu at (155.0, 160.0)
- added TP_RELAY3_CTRL1: RELAY3_CTRL, TestPoint_THTPad_1.5x1.5mm_Drill0.7mm, F.Cu at (192.0, 160.0)
- added TP_RELAY4_CTRL1: RELAY4_CTRL, TestPoint_THTPad_1.5x1.5mm_Drill0.7mm, F.Cu at (229.0, 160.0)
- added TP_RELAY5_CTRL1: RELAY5_CTRL, TestPoint_THTPad_1.5x1.5mm_Drill0.7mm, F.Cu at (266.0, 160.0)
- added TP_RELAY_GND1: GND, TestPoint_THTPad_1.5x1.5mm_Drill0.7mm, F.Cu at (100.0, 214.0)
- added TP_RELAY_PWR1: RELAY_PWR, TestPoint_THTPad_1.5x1.5mm_Drill0.7mm, F.Cu at (100.0, 208.0)
- added TP_RS485_A1: RS485_A, TestPoint_THTPad_1.5x1.5mm_Drill0.7mm, F.Cu at (68.0, 134.0)
- added TP_RS485_B1: RS485_B, TestPoint_THTPad_1.5x1.5mm_Drill0.7mm, F.Cu at (73.0, 134.0)
- added TP_RS485_DERE1: RS485_DE_RE, TestPoint_THTPad_1.5x1.5mm_Drill0.7mm, F.Cu at (78.0, 134.0)
- added TP_RS485_RX1: RS485_RX, TestPoint_THTPad_1.5x1.5mm_Drill0.7mm, F.Cu at (83.0, 134.0)
- added TP_RS485_TX1: RS485_TX, TestPoint_THTPad_1.5x1.5mm_Drill0.7mm, F.Cu at (88.0, 134.0)
- added TP_SOLAR1: SOL_PROT, TestPoint_THTPad_1.5x1.5mm_Drill0.7mm, F.Cu at (70.0, 32.0)
- added TP_USER_BTN1: USER_BTN, TestPoint_THTPad_1.5x1.5mm_Drill0.7mm, F.Cu at (257.0, 150.0)
- added U_CHG1: BQ25798_substitutes_BQ25792, Texas_RQM0029A_VQFN-29_4x4mm_P0.4mm, F.Cu at (45.0, 72.0)
- added U_LORA1: RAK3172-IN865, RAK3172, F.Cu at (245.0, 50.0)
- added U_MCU1: STM32L462RETx, LQFP-64_10x10mm_P0.5mm, F.Cu at (150.0, 120.0)
- added U_PROT1: BQ76920PW, TSSOP-20_4.4x6.5mm_P0.65mm, F.Cu at (165.0, 55.0)
- added U_RS485_1: THVD1450D, SOIC-8_3.9x4.9mm_P1.27mm, F.Cu at (75.0, 105.0)
- added Y_LSE1: 32.768kHz, Crystal_SMD_3215-2Pin_3.2x1.5mm, F.Cu at (178.0, 118.0)
- C_BST1, C_FF1, C_SS1: footprint Capacitor_SMD:C_0603_1608Metric -> C_0603_1608Metric
- C_INTVCC1: footprint Capacitor_SMD:C_0805_2012Metric -> C_0805_2012Metric
- Cin1, Cin2: footprint Capacitor_SMD:C_1210_3225Metric -> C_1210_3225Metric
- Cout1, Cout2: footprint Capacitor_SMD:C_1206_3216Metric -> C_1206_3216Metric
- D1: footprint Diode_SMD:D_SMB -> D_SMB
- D_LED1: footprint LED_SMD:LED_0805_2012Metric -> LED_0805_2012Metric
- F1: footprint Fuse:Fuse_1812_4532Metric -> Fuse_1812_4532Metric
- J1: footprint TerminalBlock_Phoenix:TerminalBlock_Phoenix_MKDS-3-2-5.08_1x02_P5.08mm_Horizontal -> TerminalBlock_Phoenix_MKDS-3-2-5.08_1x02_P5.08mm_Horizontal
- L1: footprint Inductor_SMD:L_10.4x10.4_H4.8 -> L_10.4x10.4_H4.8
- Q1: footprint Package_TO_SOT_SMD:TO-252-2 -> TO-252-2
- R1, R2, R_EN_BOT1, R_EN_TOP1, R_LED1, R_PG1, R_RT1, R_gate1: footprint Resistor_SMD:R_0805_2012Metric -> R_0805_2012Metric
- TP1, TP2, TP3, TP4: footprint TestPoint:TestPoint_THTPad_1.5x1.5mm_Drill0.7mm -> TestPoint_THTPad_1.5x1.5mm_Drill0.7mm
- U1: footprint Package_SO:MSOP-16-1EP_3x4.039mm_P0.5mm_EP1.651x2.845mm_ThermalVias -> MSOP-16-1EP_3x4.039mm_P0.5mm_EP1.651x2.845mm_ThermalVias
- moved R_PG1 117.4 mm to (118.0, 32.0)
- moved R_LED1 111.2 mm to (110.0, 38.0)
- moved C_FF1 103.6 mm to (105.0, 32.0)
- moved R_EN_BOT1 103.1 mm to (100.0, 38.0)
- moved R2 102.2 mm to (100.0, 32.0)
- moved TP4 101.0 mm to (118.0, 38.0)
- moved R1 98.3 mm to (95.0, 32.0)
- moved R_EN_TOP1 97.5 mm to (95.0, 38.0)
- moved Cout2 90.0 mm to (118.0, 22.0)
- moved Cout1 89.9 mm to (118.0, 16.0)
- moved C_BST1 88.8 mm to (90.0, 32.0)
- moved L1 87.2 mm to (108.0, 22.0)
- moved U1 87.1 mm to (95.0, 22.0)
- moved R_RT1 84.4 mm to (85.0, 32.0)
- moved C_SS1 83.9 mm to (85.0, 38.0)
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Connections:
- C_BST1 pad 2: GND -> Net-(C_BST1-Pad2)
- D_LED1 pad 2: GND -> Net-(D_LED1-A)
- L1 pad 2: GND -> Net-(C_BST1-Pad2)
- Q1 pad 1: /VIN_PROT -> Net-(Q1-G)
- R_LED1 pad 2: GND -> Net-(D_LED1-A)
- R_gate1 pad 1: unconnected-(R_gate1-Pad1) -> /VIN_PROT
- R_gate1 pad 2: unconnected-(R_gate1-Pad2) -> Net-(Q1-G)
- U1 pad 10: GND -> Net-(C_BST1-Pad2)
- U1 pad 11: GND -> Net-(C_BST1-Pad2)
- U1 pad 5: /VIN_PROT -> /VSYS
- U1 pad 6: /VIN_PROT -> /VSYS
- U1 pad 9: GND -> Net-(C_BST1-Pad2)
Other:
- board size 2147.5 x 2147.5 mm -> 300 x 220 mm
- copper layers 2 -> 4
