File: Hardware/SWAFarmNodeV1/SWAFarmNodeV1.kicad_pcb (KiCad board)
At the start: 4 copper layers, 385 x 317 mm, 165 parts, among them J1 M12_5P_A_Coded_PowerIn, Q1 IPD50N06S4L-16, U1 TPS26600PWP, U2 TPS54561, U3 TPS563201

Commit message: updated
Parts:
- removed the CMC_RS485_1 at (26.0, 189.0)
- removed the CMC_RS485_2 at (60.0, 189.0)
- removed the C_BOOT1 at (14.0, 14.0)
- removed the C_BOOT2 at (24.0, 14.0)
- removed the C_BULK2 at (14.0, 56.0)
- removed the C_COMP1 at (34.0, 14.0)
- removed the C_DEC1 at (24.0, 56.0)
- removed the C_DEC10 at (34.0, 56.0)
- removed the C_DEC2 at (44.0, 56.0)
- removed the C_DEC3 at (54.0, 56.0)
- removed the C_DEC4 at (64.0, 56.0)
- removed the C_DEC5 at (74.0, 56.0)
- removed the C_DEC6 at (84.0, 56.0)
- removed the C_DEC7 at (94.0, 56.0)
- removed the C_DEC8 at (104.0, 56.0)
- removed the C_DEC9 at (114.0, 56.0)
- removed the C_DVDT1 at (44.0, 14.0)
- removed the C_EN1 at (124.0, 56.0)
- removed the C_FILT1 at (14.0, 216.0)
- removed the C_FILT2 at (24.0, 216.0)
- removed the C_FILT3 at (34.0, 216.0)
- removed the C_FILT4 at (44.0, 216.0)
- removed the C_FILT5 at (54.0, 216.0)
- removed the C_FILT6 at (64.0, 216.0)
- removed the C_IN1 at (54.0, 14.0)
- removed the C_IN2 at (64.0, 14.0)
- removed the C_IN3 at (74.0, 14.0)
- removed the C_ISOIN1 at (82.0, 184.0)
- removed the C_ISOOUT1 at (92.0, 184.0)
- removed the C_OUT1 at (84.0, 14.0)
- removed the C_OUT2 at (94.0, 14.0)
- removed the C_OUT3 at (104.0, 14.0)
- removed the C_SS1 at (114.0, 14.0)
- removed the C_VALVEBULK1 at (18.0, 258.0)
- removed the C_VMDEC1 at (32.0, 254.0)
- removed the C_VMDEC2 at (42.0, 254.0)
- removed the C_VMDEC3 at (52.0, 254.0)
- removed the C_VMDEC4 at (62.0, 254.0)
- removed the C_VMDEC5 at (72.0, 254.0)
- removed the C_VMDEC6 at (82.0, 254.0)
- removed the D1 at (124.0, 14.0)
- removed the D_CLHI1 at (74.0, 216.0)
- removed the D_CLHI2 at (84.0, 216.0)
- removed the D_CLHI3 at (94.0, 216.0)
- removed the D_CLHI4 at (104.0, 216.0)
- removed the D_CLHI5 at (114.0, 216.0)
- removed the D_CLHI6 at (124.0, 216.0)
- removed the D_CLLO1 at (134.0, 216.0)
- removed the D_CLLO2 at (144.0, 216.0)
- removed the D_CLLO3 at (154.0, 216.0)
- removed the D_CLLO4 at (164.0, 216.0)
- removed the D_CLLO5 at (174.0, 216.0)
- removed the D_CLLO6 at (184.0, 216.0)
- removed the D_FLT1 at (14.0, 118.0)
- removed the D_LED1 at (134.0, 14.0)
- removed the D_LED2 at (144.0, 14.0)
- removed the D_LINK1 at (24.0, 118.0)
- removed the D_PWR1 at (34.0, 118.0)
- removed the D_RS485PROT1 at (102.0, 184.0)
- removed the D_RS485PROT2 at (112.0, 184.0)
- removed the F1 at (154.0, 14.0)
- removed the J1 at (174.0, 21.0)
- removed the J_LORASMA1 at (24.0, 145.0)
- removed the J_OUT1 at (204.0, 21.0)
- removed the J_PROG1 at (144.0, 63.0)
- removed the J_RS485_IN1 at (132.0, 191.0)
- removed the J_RS485_LOC1 at (162.0, 191.0)
- removed the J_RS485_OUT1 at (192.0, 191.0)
- removed the J_SENSOR_RET1 at (219.0, 221.0)
- removed the J_SENSOR_SIG1 at (279.0, 221.0)
- removed the J_USB1 at (174.0, 63.0)
- removed the J_VALVE_OUT1_1 at (117.0, 259.0)
- removed the J_VALVE_OUT2_1 at (177.0, 259.0)
- removed the L1 at (225.5, 15.5)
- removed the L2 at (238.5, 15.5)
- removed the Q1 at (250.0, 14.0)
- removed the R_BIASA1 at (212.0, 184.0)
- removed the R_BIASB1 at (222.0, 184.0)
- removed the R_BOOT1 at (194.0, 56.0)
- removed the R_BURDEN1 at (314.0, 216.0)
- removed the R_BURDEN2 at (324.0, 216.0)
- removed the R_BURDEN3 at (334.0, 216.0)
- removed the R_BURDEN4 at (344.0, 216.0)
- removed the R_BURDEN5 at (354.0, 216.0)
- removed the R_BURDEN6 at (364.0, 216.0)
- removed the R_CC1_1 at (204.0, 56.0)
- removed the R_CC2_1 at (214.0, 56.0)
- removed the R_COMP1 at (260.0, 14.0)
- removed the R_EN1A1 at (270.0, 14.0)
- removed the R_EN1B1 at (280.0, 14.0)
- removed the R_EN2 at (290.0, 14.0)
- removed the R_ENPU1 at (224.0, 56.0)
- removed the R_EXPRST1 at (212.0, 254.0)
- removed the R_FB1A1 at (300.0, 14.0)
- removed the R_FB1B1 at (310.0, 14.0)
- removed the R_FB2A1 at (320.0, 14.0)
- removed the R_FB2B1 at (330.0, 14.0)
- removed the R_FLT1 at (340.0, 14.0)
- removed the R_ILIM1 at (350.0, 14.0)
- removed the R_ILIM_V1 at (222.0, 254.0)
- removed the R_ILIM_V2 at (232.0, 254.0)
- removed the R_ILIM_V3 at (242.0, 254.0)
- removed the R_ILIM_V4 at (252.0, 254.0)
- removed the R_ILIM_V5 at (262.0, 254.0)
- removed the R_ILIM_V6 at (272.0, 254.0)
- removed the R_IMON1 at (360.0, 14.0)
- removed the R_LED1 at (370.0, 14.0)
- removed the R_LED2 at (14.0, 38.0)
- removed the R_LEDFLT1 at (44.0, 118.0)
- removed the R_LINK1 at (54.0, 118.0)
- removed the R_LORABOOT1 at (44.0, 138.0)
- removed the R_LORARST1 at (54.0, 138.0)
- removed the R_OVP1 at (24.0, 38.0)
- removed the R_OVP2 at (34.0, 38.0)
- removed the R_PG1 at (44.0, 38.0)
- removed the R_PWR1 at (64.0, 118.0)
- removed the R_RT1 at (54.0, 38.0)
- removed the R_SER1 at (14.0, 236.0)
- removed the R_SER2 at (24.0, 236.0)
- removed the R_SER3 at (34.0, 236.0)
- removed the R_SER4 at (44.0, 236.0)
- removed the R_SER5 at (54.0, 236.0)
- removed the R_SER6 at (64.0, 236.0)
- removed the R_SETUP1 at (74.0, 118.0)
- removed the R_SHDN1 at (64.0, 38.0)
- removed the R_TERM1 at (232.0, 184.0)
- removed the R_UVLO1 at (74.0, 38.0)
- removed the R_UVLO2 at (84.0, 38.0)
- removed the R_gate1 at (94.0, 38.0)
- removed the SW_BOOT1 at (235.0, 57.0)
- removed the SW_RESET1 at (247.0, 57.0)
- removed the SW_SETUP1 at (85.0, 119.0)
- removed the TP_12V_SW1 at (103.0, 37.0)
- removed the TP_3V3 at (111.0, 37.0)
- removed the TP_5V1 at (119.0, 37.0)
- removed the TP_FLT1 at (127.0, 37.0)
- removed the TP_GND1 at (135.0, 37.0)
- removed the TP_IMON1 at (143.0, 37.0)
- removed the TP_ISO5V1 at (241.0, 183.0)
- removed the TP_ISOGND1 at (249.0, 183.0)
- removed the TP_LORABOOT1 at (63.0, 137.0)
- removed the TP_LORARST1 at (71.0, 137.0)
- removed the TP_PG1 at (151.0, 37.0)
- removed the TP_RS485DI1 at (257.0, 183.0)
- removed the TP_RS485RO1 at (265.0, 183.0)
- removed the TP_USBVBUS1 at (257.0, 55.0)
- removed the U1 at (160.0, 38.0)
- removed the U2 at (170.0, 38.0)
- removed the U3 at (180.0, 38.0)
- removed the U_DRV1 at (286.0, 257.0)
- removed the U_DRV2 at (304.0, 257.0)
- removed the U_DRV3 at (322.0, 257.0)
- removed the U_DRV4 at (340.0, 257.0)
- removed the U_DRV5 at (358.0, 257.0)
- removed the U_DRV6 at (18.0, 277.0)
- removed the U_ISO1 at (283.0, 191.0)
- removed the U_ISODCDC1 at (311.0, 191.0)
- removed the U_LORA1 at (93.0, 152.0)
- removed the U_MCU1 at (293.0, 78.0)
- removed the U_RS485_TX1 at (334.0, 187.0)
- removed the U_VALVEEXP1 at (41.0, 281.0)
- added CMC_RS485_1: 744232090, L_CommonModeChoke_Bourns_SRF1260, F.Cu at (26.4, 197.0)
- added CMC_RS485_1: 744232090, Inductor_SMD:L_CommonModeChoke_Bourns_SRF1260, F.Cu at (368.7, 154.8)
- added CMC_RS485_2: 744232090, L_CommonModeChoke_Bourns_SRF1260, F.Cu at (61.2, 197.0)
- added CMC_RS485_2: 744232090, Inductor_SMD:L_CommonModeChoke_Bourns_SRF1260, F.Cu at (368.7, 168.8)
- added C_BOOT1: 100nF, C_0603_1608Metric, F.Cu at (19.0, 13.8)
- added C_BOOT1: 100nF, Capacitor_SMD:C_0603_1608Metric, F.Cu at (344.6, 106.8)
- added C_BOOT2: 100nF, Capacitor_SMD:C_0603_1608Metric, F.Cu at (344.6, 109.3)
- added C_BOOT2: 100nF, C_0603_1608Metric, F.Cu at (38.9, 13.8)
- added C_BULK2: 10uF, Capacitor_SMD:C_1206_3216Metric, F.Cu at (361.4, 120.6)
- added C_BULK2: 10uF, C_1206_3216Metric, F.Cu at (19.0, 66.4)
- added C_COMP1: 2.2nF_TBD, C_0603_1608Metric, F.Cu at (58.8, 13.8)
- added C_COMP1: 2.2nF_TBD, Capacitor_SMD:C_0603_1608Metric, F.Cu at (344.6, 111.8)
- added C_DEC1: 100nF, Capacitor_SMD:C_0603_1608Metric, F.Cu at (344.6, 114.3)
- added C_DEC1: 100nF, C_0603_1608Metric, F.Cu at (38.9, 65.9)
- added C_DEC10: 100nF, Capacitor_SMD:C_0603_1608Metric, F.Cu at (352.6, 106.8)
- added C_DEC10: 100nF, C_0603_1608Metric, F.Cu at (58.8, 65.9)
- added C_DEC2: 100nF, Capacitor_SMD:C_0603_1608Metric, F.Cu at (344.6, 116.8)
- added C_DEC2: 100nF, C_0603_1608Metric, F.Cu at (78.7, 65.9)
- added C_DEC3: 100nF, C_0603_1608Metric, F.Cu at (98.6, 65.9)
- added C_DEC3: 100nF, Capacitor_SMD:C_0603_1608Metric, F.Cu at (344.6, 119.3)
- added C_DEC4: 100nF, C_0603_1608Metric, F.Cu at (118.5, 65.9)
- added C_DEC4: 100nF, Capacitor_SMD:C_0603_1608Metric, F.Cu at (348.6, 106.8)
- added C_DEC5: 100nF, Capacitor_SMD:C_0603_1608Metric, F.Cu at (348.6, 109.3)
- added C_DEC5: 100nF, C_0603_1608Metric, F.Cu at (138.5, 65.9)
- added C_DEC6: 100nF, C_0603_1608Metric, F.Cu at (158.4, 65.9)
- added C_DEC6: 100nF, Capacitor_SMD:C_0603_1608Metric, F.Cu at (348.6, 111.8)
- added C_DEC7: 100nF, C_0603_1608Metric, F.Cu at (178.3, 65.9)
- added C_DEC7: 100nF, Capacitor_SMD:C_0603_1608Metric, F.Cu at (348.6, 114.3)
- added C_DEC8: 100nF, Capacitor_SMD:C_0603_1608Metric, F.Cu at (348.6, 116.8)
- added C_DEC8: 100nF, C_0603_1608Metric, F.Cu at (198.2, 65.9)
- added C_DEC9: 100nF, Capacitor_SMD:C_0603_1608Metric, F.Cu at (348.6, 119.3)
- added C_DEC9: 100nF, C_0603_1608Metric, F.Cu at (218.1, 65.9)
- added C_DVDT1: 1nF_TBD, C_0805_2012Metric, F.Cu at (78.7, 14.0)
- added C_DVDT1: 1nF_TBD, Capacitor_SMD:C_0805_2012Metric, F.Cu at (366.5, 120.4)
- added C_EN1: 1uF, C_0805_2012Metric, F.Cu at (238.0, 66.2)
- added C_EN1: 1uF, Capacitor_SMD:C_0805_2012Metric, F.Cu at (366.5, 123.4)
- added C_FILT1: 100nF, Capacitor_SMD:C_0603_1608Metric, F.Cu at (352.6, 109.3)
- added C_FILT1: 100nF, C_0603_1608Metric, F.Cu at (19.0, 242.0)
- added C_FILT2: 100nF, Capacitor_SMD:C_0603_1608Metric, F.Cu at (352.6, 111.8)
- added C_FILT2: 100nF, C_0603_1608Metric, F.Cu at (38.9, 242.0)
- added C_FILT3: 100nF, Capacitor_SMD:C_0603_1608Metric, F.Cu at (352.6, 114.3)
- added C_FILT3: 100nF, C_0603_1608Metric, F.Cu at (58.8, 242.0)
- added C_FILT4: 100nF, Capacitor_SMD:C_0603_1608Metric, F.Cu at (352.6, 116.8)
- added C_FILT4: 100nF, C_0603_1608Metric, F.Cu at (78.7, 242.0)
- added C_FILT5: 100nF, C_0603_1608Metric, F.Cu at (98.6, 242.0)
- added C_FILT5: 100nF, Capacitor_SMD:C_0603_1608Metric, F.Cu at (352.6, 119.3)
- added C_FILT6: 100nF, C_0603_1608Metric, F.Cu at (118.5, 242.0)
- added C_FILT6: 100nF, Capacitor_SMD:C_0603_1608Metric, F.Cu at (356.6, 106.8)
- added C_IN1: 10uF_25V, C_1206_3216Metric, F.Cu at (98.6, 14.2)
- added C_IN1: 10uF_25V, Capacitor_SMD:C_1206_3216Metric, F.Cu at (361.4, 123.9)
- added C_IN2: 10uF_25V, C_1206_3216Metric, F.Cu at (118.5, 14.2)
- added C_IN2: 10uF_25V, Capacitor_SMD:C_1206_3216Metric, F.Cu at (361.4, 127.3)
- added C_IN3: 10uF_16V, C_1206_3216Metric, F.Cu at (138.5, 14.2)
- added C_IN3: 10uF_16V, Capacitor_SMD:C_1206_3216Metric, F.Cu at (361.4, 130.6)
- added C_ISOIN1: 100nF, Capacitor_SMD:C_0603_1608Metric, F.Cu at (356.6, 109.3)
- added C_ISOIN1: 100nF, C_0603_1608Metric, F.Cu at (88.5, 191.2)
- added C_ISOOUT1: 100nF, Capacitor_SMD:C_0603_1608Metric, F.Cu at (356.6, 111.8)
- added C_ISOOUT1: 100nF, C_0603_1608Metric, F.Cu at (108.4, 191.2)
- added C_OUT1: 10uF_25V, C_1206_3216Metric, F.Cu at (158.4, 14.2)
- added C_OUT1: 10uF_25V, Capacitor_SMD:C_1206_3216Metric, F.Cu at (361.4, 134.0)
- added C_OUT2: 22uF_10V, C_1206_3216Metric, F.Cu at (178.3, 14.2)
- added C_OUT2: 22uF_10V, Capacitor_SMD:C_1206_3216Metric, F.Cu at (361.4, 137.3)
- added C_OUT3: 22uF_10V, Capacitor_SMD:C_1206_3216Metric, F.Cu at (361.4, 140.7)
- added C_OUT3: 22uF_10V, C_1206_3216Metric, F.Cu at (198.2, 14.2)
- added C_SS1: 10nF_TBD, C_0603_1608Metric, F.Cu at (218.1, 13.8)
- added C_SS1: 10nF_TBD, Capacitor_SMD:C_0603_1608Metric, F.Cu at (356.6, 114.3)
- added C_VALVEBULK1: 1000uF_25V, Capacitor_THT:CP_Radial_D12.5mm_P5.00mm, F.Cu at (373.6, 140.7)
- added C_VALVEBULK1: 1000uF_25V, CP_Radial_D12.5mm_P5.00mm, F.Cu at (20.6, 293.6)
- added C_VMDEC1: 1uF, C_0805_2012Metric, F.Cu at (47.2, 287.8)
- added C_VMDEC1: 1uF, Capacitor_SMD:C_0805_2012Metric, F.Cu at (366.5, 126.4)
- added C_VMDEC2: 1uF, Capacitor_SMD:C_0805_2012Metric, F.Cu at (366.5, 129.4)
- added C_VMDEC2: 1uF, C_0805_2012Metric, F.Cu at (67.1, 287.8)
- added C_VMDEC3: 1uF, Capacitor_SMD:C_0805_2012Metric, F.Cu at (366.5, 132.4)
- added C_VMDEC3: 1uF, C_0805_2012Metric, F.Cu at (87.0, 287.8)
- added C_VMDEC4: 1uF, Capacitor_SMD:C_0805_2012Metric, F.Cu at (366.5, 135.5)
- added C_VMDEC4: 1uF, C_0805_2012Metric, F.Cu at (107.0, 287.8)
- added C_VMDEC5: 1uF, Capacitor_SMD:C_0805_2012Metric, F.Cu at (366.5, 138.5)
- added C_VMDEC5: 1uF, C_0805_2012Metric, F.Cu at (126.9, 287.8)
- added C_VMDEC6: 1uF, Capacitor_SMD:C_0805_2012Metric, F.Cu at (366.5, 141.5)
- added C_VMDEC6: 1uF, C_0805_2012Metric, F.Cu at (146.8, 287.8)
- added D1: SMBJ18CA, D_SMB, F.Cu at (234.3, 15.3)
- added D1: SMBJ18CA, Diode_SMD:D_SMB, F.Cu at (380.2, 173.0)
- added D_CLHI1: BAV99_1of2, Diode_SMD:D_SOD-123, F.Cu at (361.5, 107.2)
- added D_CLHI1: BAV99_1of2, D_SOD-123, F.Cu at (135.6, 242.6)
- added D_CLHI2: BAV99_1of2, Diode_SMD:D_SOD-123, F.Cu at (361.5, 110.5)
- added D_CLHI2: BAV99_1of2, D_SOD-123, F.Cu at (149.7, 242.6)
- added D_CLHI3: BAV99_1of2, D_SOD-123, F.Cu at (163.8, 242.6)
- added D_CLHI3: BAV99_1of2, Diode_SMD:D_SOD-123, F.Cu at (361.5, 113.9)
- added D_CLHI4: BAV99_1of2, Diode_SMD:D_SOD-123, F.Cu at (361.5, 117.2)
- added D_CLHI4: BAV99_1of2, D_SOD-123, F.Cu at (177.9, 242.6)
- added D_CLHI5: BAV99_1of2, D_SOD-123, F.Cu at (192.0, 242.6)
- added D_CLHI5: BAV99_1of2, Diode_SMD:D_SOD-123, F.Cu at (367.3, 107.2)
- added D_CLHI6: BAV99_1of2, D_SOD-123, F.Cu at (206.1, 242.6)
- added D_CLHI6: BAV99_1of2, Diode_SMD:D_SOD-123, F.Cu at (367.3, 110.5)
- added D_CLLO1: BAV99_2of2, Diode_SMD:D_SOD-123, F.Cu at (367.3, 113.9)
- added D_CLLO1: BAV99_2of2, D_SOD-123, F.Cu at (220.2, 242.6)
- added D_CLLO2: BAV99_2of2, Diode_SMD:D_SOD-123, F.Cu at (367.3, 117.2)
- added D_CLLO2: BAV99_2of2, D_SOD-123, F.Cu at (234.3, 242.6)
- added D_CLLO3: BAV99_2of2, Diode_SMD:D_SOD-123, F.Cu at (373.1, 107.2)
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Other:
- board size 385 x 317 mm -> 420 x 354.9 mm

Commit message: updated
Parts:
- removed the CMC_RS485_1 at (26.4, 197.0)
- removed the CMC_RS485_1 at (368.7, 154.8)
- removed the CMC_RS485_2 at (61.2, 197.0)
- removed the CMC_RS485_2 at (368.7, 168.8)
- removed the C_BOOT1 at (344.6, 106.8)
- removed the C_BOOT2 at (344.6, 109.3)
- removed the C_BULK2 at (361.4, 120.6)
- removed the C_BULK2 at (19.0, 66.4)
- removed the C_COMP1 at (344.6, 111.8)
- removed the C_DEC1 at (344.6, 114.3)
- removed the C_DEC1 at (38.9, 65.9)
- removed the C_DEC10 at (352.6, 106.8)
- removed the C_DEC10 at (58.8, 65.9)
- removed the C_DEC2 at (344.6, 116.8)
- removed the C_DEC2 at (78.7, 65.9)
- removed the C_DEC3 at (98.6, 65.9)
- removed the C_DEC3 at (344.6, 119.3)
- removed the C_DEC4 at (118.5, 65.9)
- removed the C_DEC4 at (348.6, 106.8)
- removed the C_DEC5 at (348.6, 109.3)
- removed the C_DEC5 at (138.5, 65.9)
- removed the C_DEC6 at (158.4, 65.9)
- removed the C_DEC6 at (348.6, 111.8)
- removed the C_DEC7 at (178.3, 65.9)
- removed the C_DEC7 at (348.6, 114.3)
- removed the C_DEC8 at (348.6, 116.8)
- removed the C_DEC8 at (198.2, 65.9)
- removed the C_DEC9 at (348.6, 119.3)
- removed the C_DEC9 at (218.1, 65.9)
- removed the C_DVDT1 at (366.5, 120.4)
- removed the C_EN1 at (238.0, 66.2)
- removed the C_EN1 at (366.5, 123.4)
- removed the C_FILT1 at (352.6, 109.3)
- removed the C_FILT1 at (19.0, 242.0)
- removed the C_FILT2 at (352.6, 111.8)
- removed the C_FILT2 at (38.9, 242.0)
- removed the C_FILT3 at (352.6, 114.3)
- removed the C_FILT3 at (58.8, 242.0)
- removed the C_FILT4 at (352.6, 116.8)
- removed the C_FILT4 at (78.7, 242.0)
- removed the C_FILT5 at (98.6, 242.0)
- removed the C_FILT5 at (352.6, 119.3)
- removed the C_FILT6 at (118.5, 242.0)
- removed the C_FILT6 at (356.6, 106.8)
- removed the C_IN1 at (361.4, 123.9)
- removed the C_IN2 at (361.4, 127.3)
- removed the C_IN3 at (361.4, 130.6)
- removed the C_ISOIN1 at (356.6, 109.3)
- removed the C_ISOIN1 at (88.5, 191.2)
- removed the C_ISOOUT1 at (356.6, 111.8)
- removed the C_ISOOUT1 at (108.4, 191.2)
- removed the C_OUT1 at (361.4, 134.0)
- removed the C_OUT2 at (361.4, 137.3)
- removed the C_OUT3 at (361.4, 140.7)
- removed the C_SS1 at (356.6, 114.3)
- removed the C_VALVEBULK1 at (373.6, 140.7)
- removed the C_VALVEBULK1 at (20.6, 293.6)
- removed the C_VMDEC1 at (47.2, 287.8)
- removed the C_VMDEC1 at (366.5, 126.4)
- removed the C_VMDEC2 at (366.5, 129.4)
- removed the C_VMDEC2 at (67.1, 287.8)
- removed the C_VMDEC3 at (366.5, 132.4)
- removed the C_VMDEC3 at (87.0, 287.8)
- removed the C_VMDEC4 at (366.5, 135.5)
- removed the C_VMDEC4 at (107.0, 287.8)
- removed the C_VMDEC5 at (366.5, 138.5)
- removed the C_VMDEC5 at (126.9, 287.8)
- removed the C_VMDEC6 at (366.5, 141.5)
- removed the C_VMDEC6 at (146.8, 287.8)
- removed the D1 at (380.2, 173.0)
- removed the D_CLHI1 at (361.5, 107.2)
- removed the D_CLHI1 at (135.6, 242.6)
- removed the D_CLHI2 at (361.5, 110.5)
- removed the D_CLHI2 at (149.7, 242.6)
- removed the D_CLHI3 at (163.8, 242.6)
- removed the D_CLHI3 at (361.5, 113.9)
- removed the D_CLHI4 at (361.5, 117.2)
- removed the D_CLHI4 at (177.9, 242.6)
- removed the D_CLHI5 at (192.0, 242.6)
- removed the D_CLHI5 at (367.3, 107.2)
- removed the D_CLHI6 at (206.1, 242.6)
- removed the D_CLHI6 at (367.3, 110.5)
- removed the D_CLLO1 at (367.3, 113.9)
- removed the D_CLLO1 at (220.2, 242.6)
- removed the D_CLLO2 at (367.3, 117.2)
- removed the D_CLLO2 at (234.3, 242.6)
- removed the D_CLLO3 at (373.1, 107.2)
- removed the D_CLLO3 at (248.4, 242.6)
- removed the D_CLLO4 at (262.5, 242.6)
- removed the D_CLLO4 at (373.1, 110.5)
- removed the D_CLLO5 at (373.1, 113.9)
- removed the D_CLLO5 at (276.6, 242.6)
- removed the D_CLLO6 at (290.7, 242.6)
- removed the D_CLLO6 at (373.1, 117.2)
- removed the D_FLT1 at (19.8, 139.8)
- removed the D_FLT1 at (355.4, 122.1)
- removed the D_LED1 at (355.4, 125.1)
- removed the D_LED2 at (355.4, 128.2)
- removed the D_LINK1 at (355.4, 131.2)
- removed the D_LINK1 at (41.4, 139.8)
- removed the D_PWR1 at (63.1, 139.8)
- removed the D_PWR1 at (355.4, 134.2)
- removed the D_RS485PROT1 at (384.9, 121.1)
- removed the D_RS485PROT1 at (124.0, 192.2)
- removed the D_RS485PROT2 at (135.1, 192.2)
- removed the D_RS485PROT2 at (384.9, 125.6)
- removed the F1 at (356.0, 196.8)
- removed the J1 at (378.3, 107.8)
- removed the J1 at (321.8, 14.7)
- removed the J_LORASMA1 at (23.5, 162.6)
- removed the J_LORASMA1 at (380.7, 165.5)
- removed the J_OUT1 at (353.2, 14.7)
- removed the J_OUT1 at (382.9, 107.8)
- removed the J_PROG1 at (384.1, 150.0)
- removed the J_PROG1 at (263.7, 66.9)
- removed the J_RS485_IN1 at (371.0, 121.2)
- removed the J_RS485_IN1 at (156.4, 192.2)
- removed the J_RS485_LOC1 at (187.9, 192.2)
- removed the J_RS485_LOC1 at (375.6, 121.2)
- removed the J_RS485_OUT1 at (380.2, 121.2)
- removed the J_RS485_OUT1 at (219.3, 192.2)
- removed the J_SENSOR_RET1 at (297.1, 154.0)
- removed the J_SENSOR_RET1 at (314.2, 246.9)
- removed the J_SENSOR_SIG1 at (25.4, 265.7)
- removed the J_SENSOR_SIG1 at (297.1, 166.1)
- removed the J_USB1 at (344.8, 192.1)
- removed the J_USB1 at (298.4, 70.2)
- removed the J_VALVE_OUT1_1 at (173.2, 292.4)
- removed the J_VALVE_OUT1_1 at (297.1, 178.2)
- removed the J_VALVE_OUT2_1 at (297.1, 190.4)
- removed the J_VALVE_OUT2_1 at (231.4, 292.4)
- removed the L1 at (383.1, 192.8)
- removed the L1 at (379.0, 16.3)
- removed the L2 at (329.1, 196.6)
- removed the L2 at (399.0, 15.4)
- removed the Q1 at (14.6, 33.8)
- removed the Q1 at (384.9, 130.0)
- removed the R_BIASA1 at (245.0, 191.4)
- removed the R_BIASA1 at (328.2, 149.2)
- removed the R_BIASB1 at (328.2, 152.2)
- removed the R_BIASB1 at (264.9, 191.4)
- removed the R_BOOT1 at (328.2, 155.1)
- removed the R_BOOT1 at (327.4, 66.2)
- removed the R_BURDEN1 at (77.2, 261.0)
- removed the R_BURDEN1 at (328.2, 158.1)
- removed the R_BURDEN2 at (328.2, 161.0)
- removed the R_BURDEN2 at (97.1, 261.0)
- removed the R_BURDEN3 at (328.2, 164.0)
- removed the R_BURDEN3 at (117.0, 261.0)
- removed the R_BURDEN4 at (136.9, 261.0)
- removed the R_BURDEN4 at (328.2, 166.9)
- removed the R_BURDEN5 at (328.2, 169.9)
- removed the R_BURDEN5 at (156.8, 261.0)
- removed the R_BURDEN6 at (176.7, 261.0)
- removed the R_BURDEN6 at (328.2, 172.8)
- removed the R_CC1_1 at (332.6, 149.2)
- removed the R_CC1_1 at (347.3, 66.2)
- removed the R_CC2_1 at (332.6, 152.2)
- removed the R_CC2_1 at (367.2, 66.2)
- removed the R_COMP1 at (332.6, 155.1)
- removed the R_COMP1 at (30.1, 33.1)
- removed the R_EN1A1 at (332.6, 161.0)
- removed the R_EN1A1 at (50.0, 33.1)
- removed the R_EN1B1 at (69.9, 33.1)
- removed the R_EN1B1 at (332.6, 164.0)
- removed the R_EN2 at (89.9, 33.1)
- removed the R_EN2 at (332.6, 158.1)
- removed the R_ENPU1 at (332.6, 166.9)
- removed the R_ENPU1 at (387.2, 66.2)
- removed the R_EXPRST1 at (332.6, 169.9)
- removed the R_EXPRST1 at (283.1, 287.7)
- removed the R_FB1A1 at (109.8, 33.1)
- removed the R_FB1A1 at (332.6, 172.8)
- removed the R_FB1B1 at (129.7, 33.1)
- removed the R_FB1B1 at (337.1, 149.2)
- removed the R_FB2A1 at (149.6, 33.1)
- removed the R_FB2A1 at (337.1, 152.2)
- removed the R_FB2B1 at (169.5, 33.1)
- removed the R_FB2B1 at (337.1, 155.1)
- removed the R_FLT1 at (337.1, 158.1)
- removed the R_FLT1 at (189.4, 33.1)
- removed the R_ILIM1 at (209.4, 33.1)
- removed the R_ILIM1 at (337.1, 161.0)
- removed the R_ILIM_V1 at (337.1, 164.0)
- removed the R_ILIM_V1 at (303.0, 287.7)
- removed the R_ILIM_V2 at (322.9, 287.7)
- removed the R_ILIM_V2 at (337.1, 166.9)
- removed the R_ILIM_V3 at (342.9, 287.7)
- removed the R_ILIM_V3 at (337.1, 169.9)
- removed the R_ILIM_V4 at (362.8, 287.7)
- removed the R_ILIM_V4 at (337.1, 172.8)
- removed the R_ILIM_V5 at (382.7, 287.7)
- removed the R_ILIM_V5 at (341.5, 149.2)
- removed the R_ILIM_V6 at (341.5, 152.2)
- removed the R_ILIM_V6 at (19.0, 309.4)
- removed the R_IMON1 at (229.3, 33.1)
- removed the R_IMON1 at (341.5, 155.1)
- removed the R_LED1 at (249.2, 33.1)
- removed the R_LED1 at (341.5, 158.1)
- removed the R_LED2 at (269.1, 33.1)
- removed the R_LED2 at (341.5, 161.0)
- removed the R_LEDFLT1 at (341.5, 164.0)
- removed the R_LEDFLT1 at (83.9, 139.8)
- removed the R_LINK1 at (103.8, 139.8)
- removed the R_LINK1 at (341.5, 166.9)
- removed the R_LORABOOT1 at (341.5, 169.9)
- removed the R_LORABOOT1 at (48.0, 159.5)
- removed the R_LORARST1 at (67.9, 159.5)
- removed the R_LORARST1 at (341.5, 172.8)
- removed the R_OVP1 at (289.0, 33.1)
- removed the R_OVP1 at (345.9, 149.2)
- removed the R_OVP2 at (345.9, 152.2)
- removed the R_OVP2 at (308.9, 33.1)
- removed the R_PG1 at (345.9, 155.1)
- removed the R_PG1 at (328.9, 33.1)
- removed the R_PWR1 at (123.7, 139.8)
- removed the R_PWR1 at (345.9, 158.1)
- removed the R_RT1 at (348.8, 33.1)
- removed the R_RT1 at (345.9, 161.0)
- removed the R_SER1 at (345.9, 164.0)
- removed the R_SER1 at (196.7, 261.0)
- removed the R_SER2 at (216.6, 261.0)
- removed the R_SER2 at (345.9, 166.9)
- removed the R_SER3 at (345.9, 169.9)
- removed the R_SER3 at (236.5, 261.0)
- removed the R_SER4 at (256.4, 261.0)
- removed the R_SER4 at (345.9, 172.8)
- removed the R_SER5 at (276.3, 261.0)
- removed the R_SER5 at (350.3, 149.2)
- removed the R_SER6 at (350.3, 152.2)
- removed the R_SER6 at (296.2, 261.0)
- removed the R_SETUP1 at (143.6, 139.8)
- removed the R_SETUP1 at (350.3, 155.1)
- removed the R_SHDN1 at (368.7, 33.1)
- removed the R_SHDN1 at (350.3, 158.1)
- removed the R_TERM1 at (350.3, 161.0)
- removed the R_TERM1 at (284.8, 191.4)
- removed the R_UVLO1 at (350.3, 164.0)
- removed the R_UVLO1 at (388.6, 33.1)
- removed the R_UVLO2 at (350.3, 166.9)
- removed the R_UVLO2 at (19.0, 44.6)
- removed the R_gate1 at (350.3, 169.9)
- removed the R_gate1 at (38.9, 44.6)
- removed the SW_BOOT1 at (19.8, 84.5)
- removed the SW_BOOT1 at (378.9, 149.9)
- removed the SW_RESET1 at (41.4, 84.5)
- removed the SW_RESET1 at (378.9, 154.3)
- removed the SW_SETUP1 at (164.4, 140.7)
- removed the SW_SETUP1 at (378.9, 158.6)
- removed the TP_12V_SW1 at (344.3, 122.3)
- removed the TP_12V_SW1 at (60.1, 44.6)
- removed the TP_3V3 at (344.3, 125.9)
- removed the TP_3V3 at (82.6, 44.6)
- removed the TP_5V1 at (105.1, 44.6)
- removed the TP_5V1 at (344.3, 129.4)
- removed the TP_FLT1 at (344.3, 133.0)
- removed the TP_FLT1 at (127.5, 44.6)
- removed the TP_GND1 at (150.0, 44.6)
- removed the TP_GND1 at (344.3, 136.5)
- removed the TP_IMON1 at (172.5, 44.6)
- removed the TP_IMON1 at (347.9, 122.3)
- removed the TP_ISO5V1 at (306.0, 191.4)
- removed the TP_ISO5V1 at (347.9, 125.9)
- removed the TP_ISOGND1 at (347.9, 129.4)
- removed the TP_ISOGND1 at (328.5, 191.4)
- removed the TP_LORABOOT1 at (347.9, 133.0)
- removed the TP_LORABOOT1 at (89.1, 159.5)
- removed the TP_LORARST1 at (347.9, 136.5)
- removed the TP_LORARST1 at (111.6, 159.5)
- removed the TP_PG1 at (351.4, 122.3)
- removed the TP_PG1 at (195.0, 44.6)
- removed the TP_RS485DI1 at (351.4, 125.9)
- removed the TP_RS485DI1 at (351.0, 191.4)
- removed the TP_RS485RO1 at (373.5, 191.4)
- removed the TP_RS485RO1 at (351.4, 129.4)
- removed the TP_USBVBUS1 at (63.4, 83.6)
- removed the TP_USBVBUS1 at (351.4, 133.0)
- removed the U1 at (239.9, 46.4)
- removed the U1 at (347.4, 141.6)
- removed the U2 at (298.0, 45.9)
- removed the U2 at (355.3, 141.1)
- removed the U3 at (334.7, 196.3)
- removed the U3 at (329.1, 45.3)
- removed the U_DRV1 at (356.8, 151.1)
- removed the U_DRV1 at (43.8, 311.3)
- removed the U_DRV2 at (356.8, 157.8)
- removed the U_DRV2 at (73.4, 311.3)
- removed the U_DRV3 at (356.8, 164.5)
- removed the U_DRV3 at (103.1, 311.3)
- removed the U_DRV4 at (132.8, 311.3)
- removed the U_DRV4 at (356.8, 171.1)
- removed the U_DRV5 at (162.5, 311.3)
- removed the U_DRV5 at (356.8, 177.8)
- removed the U_DRV6 at (192.1, 311.3)
- removed the U_DRV6 at (356.8, 184.5)
- removed the U_ISO1 at (345.4, 180.3)
- removed the U_ISO1 at (24.4, 217.5)
- removed the U_ISODCDC1 at (381.2, 178.9)
- removed the U_ISODCDC1 at (56.8, 214.9)
- removed the U_LORA1 at (370.1, 184.9)
- removed the U_LORA1 at (134.1, 165.6)
- removed the U_MCU1 at (101.2, 108.9)
- removed the U_MCU1 at (318.0, 133.8)
- removed the U_RS485_TX1 at (356.7, 191.1)
- removed the U_RS485_TX1 at (90.6, 214.8)
- removed the U_VALVEEXP1 at (222.4, 317.7)
- removed the U_VALVEEXP1 at (332.5, 184.2)
- added CMC_RS485_1: 744232090, L_CommonModeChoke_Bourns_SRF1260, F.Cu at (26.4, 198.4)
- added CMC_RS485_2: 744232090, L_CommonModeChoke_Bourns_SRF1260, F.Cu at (61.2, 198.4)
- added C_BULK2: 10uF, C_1206_3216Metric, F.Cu at (19.0, 67.8)
- added C_DEC1: 100nF, C_0603_1608Metric, F.Cu at (38.9, 67.3)
- added C_DEC10: 100nF, C_0603_1608Metric, F.Cu at (58.8, 67.3)
- added C_DEC2: 100nF, C_0603_1608Metric, F.Cu at (78.7, 67.3)
- added C_DEC3: 100nF, C_0603_1608Metric, F.Cu at (98.6, 67.3)
- added C_DEC4: 100nF, C_0603_1608Metric, F.Cu at (118.5, 67.3)
- added C_DEC5: 100nF, C_0603_1608Metric, F.Cu at (138.5, 67.3)
- added C_DEC6: 100nF, C_0603_1608Metric, F.Cu at (158.4, 67.3)
- added C_DEC7: 100nF, C_0603_1608Metric, F.Cu at (178.3, 67.3)
- added C_DEC8: 100nF, C_0603_1608Metric, F.Cu at (198.2, 67.3)
- added C_DEC9: 100nF, C_0603_1608Metric, F.Cu at (218.1, 67.3)
- added C_EN1: 1uF, C_0805_2012Metric, F.Cu at (238.0, 67.6)
- added C_FILT1: 100nF, C_0603_1608Metric, F.Cu at (19.0, 243.4)
- added C_FILT2: 100nF, C_0603_1608Metric, F.Cu at (38.9, 243.4)
- added C_FILT3: 100nF, C_0603_1608Metric, F.Cu at (58.8, 243.4)
- added C_FILT4: 100nF, C_0603_1608Metric, F.Cu at (78.7, 243.4)
- added C_FILT5: 100nF, C_0603_1608Metric, F.Cu at (98.6, 243.4)
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Other:
- board size 420 x 354.9 mm -> 420 x 361.6 mm

Commit message: updated
Parts:
- added CMC_RS485_1: 744232090, Inductor_SMD:L_CommonModeChoke_Bourns_SRF1260, F.Cu at (555.6, 65.8)
- added CMC_RS485_2: 744232090, Inductor_SMD:L_CommonModeChoke_Bourns_SRF1260, F.Cu at (555.6, 79.8)
- added C_BOOT1: 100nF, Capacitor_SMD:C_0603_1608Metric, F.Cu at (561.5, 35.9)
- added C_BOOT2: 100nF, Capacitor_SMD:C_0603_1608Metric, F.Cu at (561.5, 38.4)
- added C_BULK2: 10uF, Capacitor_SMD:C_1206_3216Metric, F.Cu at (578.4, 36.3)
- added C_COMP1: 2.2nF_TBD, Capacitor_SMD:C_0603_1608Metric, F.Cu at (561.5, 40.9)
- added C_DEC1: 100nF, Capacitor_SMD:C_0603_1608Metric, F.Cu at (561.5, 43.4)
- added C_DEC10: 100nF, Capacitor_SMD:C_0603_1608Metric, F.Cu at (569.5, 35.9)
- added C_DEC2: 100nF, Capacitor_SMD:C_0603_1608Metric, F.Cu at (561.5, 45.9)
- added C_DEC3: 100nF, Capacitor_SMD:C_0603_1608Metric, F.Cu at (561.5, 48.4)
- added C_DEC4: 100nF, Capacitor_SMD:C_0603_1608Metric, F.Cu at (565.5, 35.9)
- added C_DEC5: 100nF, Capacitor_SMD:C_0603_1608Metric, F.Cu at (565.5, 38.4)
- added C_DEC6: 100nF, Capacitor_SMD:C_0603_1608Metric, F.Cu at (565.5, 40.9)
- added C_DEC7: 100nF, Capacitor_SMD:C_0603_1608Metric, F.Cu at (565.5, 43.4)
- added C_DEC8: 100nF, Capacitor_SMD:C_0603_1608Metric, F.Cu at (565.5, 45.9)
- added C_DEC9: 100nF, Capacitor_SMD:C_0603_1608Metric, F.Cu at (565.5, 48.4)
- added C_DVDT1: 1nF_TBD, Capacitor_SMD:C_0805_2012Metric, F.Cu at (583.4, 36.1)
- added C_EN1: 1uF, Capacitor_SMD:C_0805_2012Metric, F.Cu at (583.4, 39.2)
- added C_FILT1: 100nF, Capacitor_SMD:C_0603_1608Metric, F.Cu at (569.5, 38.4)
- added C_FILT2: 100nF, Capacitor_SMD:C_0603_1608Metric, F.Cu at (569.5, 40.9)
- added C_FILT3: 100nF, Capacitor_SMD:C_0603_1608Metric, F.Cu at (569.5, 43.4)
- added C_FILT4: 100nF, Capacitor_SMD:C_0603_1608Metric, F.Cu at (569.5, 45.9)
- added C_FILT5: 100nF, Capacitor_SMD:C_0603_1608Metric, F.Cu at (569.5, 48.4)
- added C_FILT6: 100nF, Capacitor_SMD:C_0603_1608Metric, F.Cu at (573.5, 35.9)
- added C_IN1: 10uF_25V, Capacitor_SMD:C_1206_3216Metric, F.Cu at (578.4, 39.7)
- added C_IN2: 10uF_25V, Capacitor_SMD:C_1206_3216Metric, F.Cu at (578.4, 43.0)
- added C_IN3: 10uF_16V, Capacitor_SMD:C_1206_3216Metric, F.Cu at (578.4, 46.4)
- added C_ISOIN1: 100nF, Capacitor_SMD:C_0603_1608Metric, F.Cu at (573.5, 38.4)
- added C_ISOOUT1: 100nF, Capacitor_SMD:C_0603_1608Metric, F.Cu at (573.5, 40.9)
- added C_OUT1: 10uF_25V, Capacitor_SMD:C_1206_3216Metric, F.Cu at (578.4, 49.7)
- added C_OUT2: 22uF_10V, Capacitor_SMD:C_1206_3216Metric, F.Cu at (578.4, 53.1)
- added C_OUT3: 22uF_10V, Capacitor_SMD:C_1206_3216Metric, F.Cu at (578.4, 56.4)
- added C_SS1: 10nF_TBD, Capacitor_SMD:C_0603_1608Metric, F.Cu at (573.5, 43.4)
- added C_VALVEBULK1: 1000uF_25V, Capacitor_THT:CP_Radial_D12.5mm_P5.00mm, F.Cu at (566.6, 93.9)
- added C_VMDEC1: 1uF, Capacitor_SMD:C_0805_2012Metric, F.Cu at (583.4, 42.2)
- added C_VMDEC2: 1uF, Capacitor_SMD:C_0805_2012Metric, F.Cu at (583.4, 45.2)
- added C_VMDEC3: 1uF, Capacitor_SMD:C_0805_2012Metric, F.Cu at (583.4, 48.2)
- added C_VMDEC4: 1uF, Capacitor_SMD:C_0805_2012Metric, F.Cu at (583.4, 51.2)
- added C_VMDEC5: 1uF, Capacitor_SMD:C_0805_2012Metric, F.Cu at (583.4, 54.2)
- added C_VMDEC6: 1uF, Capacitor_SMD:C_0805_2012Metric, F.Cu at (583.4, 57.2)
- added D1: SMBJ18CA, Diode_SMD:D_SMB, F.Cu at (575.6, 82.9)
- added D_CLHI1: BAV99_1of2, Diode_SMD:D_SOD-123, F.Cu at (567.7, 18.2)
- added D_CLHI2: BAV99_1of2, Diode_SMD:D_SOD-123, F.Cu at (567.7, 21.5)
- added D_CLHI3: BAV99_1of2, Diode_SMD:D_SOD-123, F.Cu at (567.7, 24.9)
- added D_CLHI4: BAV99_1of2, Diode_SMD:D_SOD-123, F.Cu at (567.7, 28.2)
- added D_CLHI5: BAV99_1of2, Diode_SMD:D_SOD-123, F.Cu at (573.5, 18.2)
- added D_CLHI6: BAV99_1of2, Diode_SMD:D_SOD-123, F.Cu at (573.5, 21.5)
- added D_CLLO1: BAV99_2of2, Diode_SMD:D_SOD-123, F.Cu at (573.5, 24.9)
- added D_CLLO2: BAV99_2of2, Diode_SMD:D_SOD-123, F.Cu at (573.5, 28.2)
- added D_CLLO3: BAV99_2of2, Diode_SMD:D_SOD-123, F.Cu at (579.2, 18.2)
- added D_CLLO4: BAV99_2of2, Diode_SMD:D_SOD-123, F.Cu at (579.2, 21.5)
- added D_CLLO5: BAV99_2of2, Diode_SMD:D_SOD-123, F.Cu at (579.2, 24.9)
- added D_CLLO6: BAV99_2of2, Diode_SMD:D_SOD-123, F.Cu at (579.2, 28.2)
- added D_FLT1: Red_FAULT, LED_SMD:LED_0805_2012Metric, F.Cu at (583.5, 60.3)
- added D_LED1: Green_PowerGood, LED_SMD:LED_0805_2012Metric, F.Cu at (583.5, 63.3)
- added D_LED2: Green_3V3Present, LED_SMD:LED_0805_2012Metric, F.Cu at (583.5, 66.3)
- added D_LINK1: Yellow_LINK, LED_SMD:LED_0805_2012Metric, F.Cu at (583.5, 69.4)
- added D_PWR1: Green_PWR, LED_SMD:LED_0805_2012Metric, F.Cu at (583.5, 72.4)
- added D_RS485PROT1: SM712-02HTG, Package_TO_SOT_SMD:SOT-23, F.Cu at (578.6, 89.1)
- added D_RS485PROT2: SM712-02HTG, Package_TO_SOT_SMD:SOT-23, F.Cu at (578.6, 93.5)
- added F1: Polyfuse_5A, Fuse:Fuse_1812_4532Metric, F.Cu at (536.7, 90.7)
- added F2: Polyfuse_4A, Fuse:Fuse_1812_4532Metric, F.Cu at (536.7, 95.7)
- added J1: M12_5P_A_Coded_PowerIn, Connector_PinHeader_2.54mm:PinHeader_1x04_P2.54mm_Vertical, F.Cu at (523.8, 101.0)
- added JP_IGND1: I_mode_gnd, Connector_PinHeader_2.54mm:PinHeader_1x02_P2.54mm_Vertical, F.Cu at (565.2, 61.0)
- added JP_IGND2: I_mode_gnd, Connector_PinHeader_2.54mm:PinHeader_1x02_P2.54mm_Vertical, F.Cu at (569.8, 61.0)
- added JP_IGND3: I_mode_gnd, Connector_PinHeader_2.54mm:PinHeader_1x02_P2.54mm_Vertical, F.Cu at (574.4, 61.0)
- added JP_IGND4: I_mode_gnd, Connector_PinHeader_2.54mm:PinHeader_1x02_P2.54mm_Vertical, F.Cu at (579.0, 61.0)
- added JP_IGND5: I_mode_gnd, Connector_PinHeader_2.54mm:PinHeader_1x02_P2.54mm_Vertical, F.Cu at (565.2, 68.2)
- added JP_IGND6: I_mode_gnd, Connector_PinHeader_2.54mm:PinHeader_1x02_P2.54mm_Vertical, F.Cu at (569.8, 68.2)
- added JP_VBYP1: V_mode_bypass, Connector_PinHeader_2.54mm:PinHeader_1x02_P2.54mm_Vertical, F.Cu at (574.4, 68.2)
- added JP_VBYP2: V_mode_bypass, Connector_PinHeader_2.54mm:PinHeader_1x02_P2.54mm_Vertical, F.Cu at (579.0, 68.2)
- added JP_VBYP3: V_mode_bypass, Connector_PinHeader_2.54mm:PinHeader_1x02_P2.54mm_Vertical, F.Cu at (565.2, 75.3)
- added JP_VBYP4: V_mode_bypass, Connector_PinHeader_2.54mm:PinHeader_1x02_P2.54mm_Vertical, F.Cu at (569.8, 75.3)
- added JP_VBYP5: V_mode_bypass, Connector_PinHeader_2.54mm:PinHeader_1x02_P2.54mm_Vertical, F.Cu at (574.4, 75.3)
- added JP_VBYP6: V_mode_bypass, Connector_PinHeader_2.54mm:PinHeader_1x02_P2.54mm_Vertical, F.Cu at (579.0, 75.3)
- added J_LORASMA1: SMA_Bulkhead_Antenna, Connector_Coaxial:SMA_Amphenol_132134_Vertical, F.Cu at (543.2, 103.4)
- added J_OUT1: M12_5P_A_Coded_PowerOut, Connector_PinHeader_2.54mm:PinHeader_1x04_P2.54mm_Vertical, F.Cu at (528.4, 101.0)
- added J_PROG1: Debug_UART_TX_RX_GND, Connector_PinHeader_2.54mm:PinHeader_1x03_P2.54mm_Vertical, F.Cu at (583.4, 89.1)
- added J_RS485_IN1: M12_5P_A_Coded_RS485_Bus_In, Connector_PinHeader_2.54mm:PinHeader_1x05_P2.54mm_Vertical, F.Cu at (550.3, 89.1)
- added J_RS485_LOC1: M12_5P_A_Coded_RS485_Local, Connector_PinHeader_2.54mm:PinHeader_1x05_P2.54mm_Vertical, F.Cu at (554.9, 89.1)
- added J_RS485_OUT1: M12_5P_A_Coded_RS485_Bus_Out, Connector_PinHeader_2.54mm:PinHeader_1x05_P2.54mm_Vertical, F.Cu at (559.5, 89.1)
- added J_SENSOR_RET1: SensorReturn_x6, TerminalBlock_Phoenix:TerminalBlock_Phoenix_MKDS-1,5-6-5.08_1x06_P5.08mm_Horizontal, F.Cu at (492.6, 65.0)
- added J_SENSOR_SIG1: SensorSignal_x6, TerminalBlock_Phoenix:TerminalBlock_Phoenix_MKDS-1,5-6-5.08_1x06_P5.08mm_Horizontal, F.Cu at (492.6, 77.1)
- added J_USB1: USB-C_Programming, Connector_USB:USB_C_Receptacle_HRO_TYPE-C-31-M-12, F.Cu at (527.4, 94.0)
- added J_VALVE_OUT1_1: ValveOut1_x6, TerminalBlock_Phoenix:TerminalBlock_Phoenix_MKDS-1,5-6-5.08_1x06_P5.08mm_Horizontal, F.Cu at (492.6, 89.2)
- added J_VALVE_OUT2_1: ValveOut2_x6, TerminalBlock_Phoenix:TerminalBlock_Phoenix_MKDS-1,5-6-5.08_1x06_P5.08mm_Horizontal, F.Cu at (492.6, 101.4)
- added L1: 3.3uH_TBD, Inductor_SMD:L_Bourns-SRN6028, F.Cu at (563.5, 53.5)
- added L2: 2.2uH_TBD, Inductor_SMD:L_Bourns-SRN4018, F.Cu at (543.2, 91.0)
- added Q1: IPD50N06S4L-16, Package_TO_SOT_SMD:SOT-23, F.Cu at (578.6, 98.0)
- added R_BIASA1: 680, Resistor_SMD:R_0805_2012Metric, F.Cu at (523.7, 60.2)
- added R_BIASB1: 680, Resistor_SMD:R_0805_2012Metric, F.Cu at (523.7, 63.2)
- added R_BOOT1: 10k, Resistor_SMD:R_0805_2012Metric, F.Cu at (523.7, 66.1)
- added R_BURDEN1: 150_0.1pct, Resistor_SMD:R_0805_2012Metric, F.Cu at (523.7, 69.1)
- added R_BURDEN2: 150_0.1pct, Resistor_SMD:R_0805_2012Metric, F.Cu at (523.7, 72.0)
- added R_BURDEN3: 150_0.1pct, Resistor_SMD:R_0805_2012Metric, F.Cu at (523.7, 75.0)
- added R_BURDEN4: 150_0.1pct, Resistor_SMD:R_0805_2012Metric, F.Cu at (523.7, 77.9)
- added R_BURDEN5: 150_0.1pct, Resistor_SMD:R_0805_2012Metric, F.Cu at (523.7, 80.9)
- added R_BURDEN6: 150_0.1pct, Resistor_SMD:R_0805_2012Metric, F.Cu at (523.7, 83.8)
- added R_CC1_1: 5.1k, Resistor_SMD:R_0805_2012Metric, F.Cu at (523.7, 86.8)
- added R_CC2_1: 5.1k, Resistor_SMD:R_0805_2012Metric, F.Cu at (528.1, 60.2)
- added R_COMP1: 10k_TBD, Resistor_SMD:R_0805_2012Metric, F.Cu at (528.1, 63.2)
- added R_EN1A1: 73.2k_TBD, Resistor_SMD:R_0805_2012Metric, F.Cu at (528.1, 69.1)
- added R_EN1B1: 10k, Resistor_SMD:R_0805_2012Metric, F.Cu at (528.1, 72.0)
- added R_EN2: 100k, Resistor_SMD:R_0805_2012Metric, F.Cu at (528.1, 66.1)
- added R_ENPU1: 10k, Resistor_SMD:R_0805_2012Metric, F.Cu at (528.1, 75.0)
- added R_EXPRST1: 10k, Resistor_SMD:R_0805_2012Metric, F.Cu at (528.1, 77.9)
- added R_FB1A1: 52.3k, Resistor_SMD:R_0805_2012Metric, F.Cu at (528.1, 80.9)
- added R_FB1B1: 10k, Resistor_SMD:R_0805_2012Metric, F.Cu at (528.1, 83.8)
- added R_FB2A1: 32.4k, Resistor_SMD:R_0805_2012Metric, F.Cu at (528.1, 86.8)
- added R_FB2B1: 10k, Resistor_SMD:R_0805_2012Metric, F.Cu at (532.6, 60.2)
- added R_FLT1: 10k, Resistor_SMD:R_0805_2012Metric, F.Cu at (532.6, 63.2)
- added R_ILIM1: 20k_TBD, Resistor_SMD:R_0805_2012Metric, F.Cu at (532.6, 66.1)
- added R_ILIM_V1: 20k_TBD, Resistor_SMD:R_0805_2012Metric, F.Cu at (532.6, 69.1)
- added R_ILIM_V2: 20k_TBD, Resistor_SMD:R_0805_2012Metric, F.Cu at (532.6, 72.0)
- added R_ILIM_V3: 20k_TBD, Resistor_SMD:R_0805_2012Metric, F.Cu at (532.6, 75.0)
- added R_ILIM_V4: 20k_TBD, Resistor_SMD:R_0805_2012Metric, F.Cu at (532.6, 77.9)
- added R_ILIM_V5: 20k_TBD, Resistor_SMD:R_0805_2012Metric, F.Cu at (532.6, 80.9)
- added R_ILIM_V6: 20k_TBD, Resistor_SMD:R_0805_2012Metric, F.Cu at (532.6, 83.8)
- added R_IMON1: 10k, Resistor_SMD:R_0805_2012Metric, F.Cu at (532.6, 86.8)
- added R_LED1: 1k, Resistor_SMD:R_0805_2012Metric, F.Cu at (537.0, 60.2)
- added R_LED2: 330, Resistor_SMD:R_0805_2012Metric, F.Cu at (537.0, 63.2)
- added R_LEDFLT1: 1k, Resistor_SMD:R_0805_2012Metric, F.Cu at (537.0, 66.1)
- added R_LINK1: 1k, Resistor_SMD:R_0805_2012Metric, F.Cu at (537.0, 69.1)
- added R_LORABOOT1: 10k, Resistor_SMD:R_0805_2012Metric, F.Cu at (537.0, 72.0)
- added R_LORARST1: 10k, Resistor_SMD:R_0805_2012Metric, F.Cu at (537.0, 75.0)
- added R_OVP1: 124k, Resistor_SMD:R_0805_2012Metric, F.Cu at (537.0, 77.9)
- added R_OVP2: 10k, Resistor_SMD:R_0805_2012Metric, F.Cu at (537.0, 80.9)
- added R_PG1: 10k, Resistor_SMD:R_0805_2012Metric, F.Cu at (537.0, 83.8)
- added R_PWR1: 1k, Resistor_SMD:R_0805_2012Metric, F.Cu at (537.0, 86.8)
- added R_RT1: 100k_TBD, Resistor_SMD:R_0805_2012Metric, F.Cu at (541.4, 60.2)
- added R_SER1: 232k, Resistor_SMD:R_0805_2012Metric, F.Cu at (541.4, 63.2)
- added R_SER2: 232k, Resistor_SMD:R_0805_2012Metric, F.Cu at (541.4, 66.1)
- added R_SER3: 232k, Resistor_SMD:R_0805_2012Metric, F.Cu at (541.4, 69.1)
- added R_SER4: 232k, Resistor_SMD:R_0805_2012Metric, F.Cu at (541.4, 72.0)
- added R_SER5: 232k, Resistor_SMD:R_0805_2012Metric, F.Cu at (541.4, 75.0)
- added R_SER6: 232k, Resistor_SMD:R_0805_2012Metric, F.Cu at (541.4, 77.9)
- added R_SETUP1: 10k, Resistor_SMD:R_0805_2012Metric, F.Cu at (541.4, 80.9)
- added R_SHDN1: 100k, Resistor_SMD:R_0805_2012Metric, F.Cu at (541.4, 83.8)
- added R_TERM1: 120_SOLDER_SELECT, Resistor_SMD:R_0805_2012Metric, F.Cu at (541.4, 86.8)
- added R_UVLO1: 64.9k, Resistor_SMD:R_0805_2012Metric, F.Cu at (545.8, 60.2)
- added R_UVLO2: 10k, Resistor_SMD:R_0805_2012Metric, F.Cu at (545.8, 63.2)
- added R_VBOT1: 100k, Resistor_SMD:R_0805_2012Metric, F.Cu at (545.8, 66.1)
- added R_VBOT2: 100k, Resistor_SMD:R_0805_2012Metric, F.Cu at (545.8, 69.1)
- added R_VBOT3: 100k, Resistor_SMD:R_0805_2012Metric, F.Cu at (545.8, 72.0)
- added R_VBOT4: 100k, Resistor_SMD:R_0805_2012Metric, F.Cu at (545.8, 75.0)
- added R_VBOT5: 100k, Resistor_SMD:R_0805_2012Metric, F.Cu at (545.8, 77.9)
- added R_VBOT6: 100k, Resistor_SMD:R_0805_2012Metric, F.Cu at (545.8, 80.9)
- added R_gate1: 10k, Resistor_SMD:R_0805_2012Metric, F.Cu at (545.8, 83.8)
- added SW_BOOT1: BOOT, Button_Switch_SMD:SW_SPST_B3U-1000P, F.Cu at (582.4, 103.1)
- added SW_RESET1: RESET, Button_Switch_SMD:SW_SPST_B3U-1000P, F.Cu at (582.4, 107.4)
- added SW_SETUP1: SETUP, Button_Switch_SMD:SW_SPST_B3U-1000P, F.Cu at (582.4, 111.8)
- added TP_12V_SW1: V12_SW, TestPoint:TestPoint_Pad_D1.5mm, F.Cu at (563.5, 102.7)
- added TP_3V3: V3V3_RAIL, TestPoint:TestPoint_Pad_D1.5mm, F.Cu at (563.5, 106.2)
- added TP_5V1: V5_RAIL, TestPoint:TestPoint_Pad_D1.5mm, F.Cu at (563.5, 109.8)
- added TP_FLT1: nFLT, TestPoint:TestPoint_Pad_D1.5mm, F.Cu at (567.1, 102.7)
- added TP_GND1: GND, TestPoint:TestPoint_Pad_D1.5mm, F.Cu at (567.1, 106.2)
- added TP_IMON1: IMON, TestPoint:TestPoint_Pad_D1.5mm, F.Cu at (567.1, 109.8)
- added TP_ISO5V1: ISO_5V, TestPoint:TestPoint_Pad_D1.5mm, F.Cu at (570.6, 102.7)
- added TP_ISOGND1: ISO_GND, TestPoint:TestPoint_Pad_D1.5mm, F.Cu at (570.6, 106.2)
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