File: Hardware/SWAFarmNodeV1/SWAFarmNodeV1.kicad_sch (KiCad schematic)
At the start: 161 parts, among them J1 M12_5P_A_Coded_PowerIn, Q1 IPD50N06S4L-16, U1 TPS26600PWP, U2 TPS54561, U3 TPS563201

Commit message: updated
Parts:
- removed J_USB1: USB-C_Programming, Connector_USB:USB_C_Receptacle_HRO_TYPE-C-31-M-12, symbol Connector:USB_C_Receptacle_USB2.0_14P
- added J_USB1: USB-C_Programming, Connector_USB:USB_C_Receptacle_HRO_TYPE-C-31-M-12, symbol Connector:USB_C_Receptacle_16P
- J_LORASMA1, R_LORABOOT1, R_LORARST1, TP_LORABOOT1, TP_LORARST1, U_LORA1: now fitted
- U_DRV1, U_DRV2, U_DRV3, U_DRV4, U_DRV5, U_DRV6: footprint Package_SO:SOIC-8_3.9x4.9mm_P1.27mm -> Package_SO:TI_SO-PowerPAD-8_ThermalVias
Connections:
- net GND: now also J_USB1.A1 (GND), J_USB1.A12 (GND), J_USB1.B1 (GND), J_USB1.B12 (GND), J_USB1.SH (SHIELD)
- net net_CC1: now also J_USB1.A5 (CC1)
- net net_CC2: now also J_USB1.B5 (CC2)
- net net_USB_DM: now also J_USB1.A7 (D-), J_USB1.B7 (D-)
- net net_USB_DP: now also J_USB1.A6 (D+), J_USB1.B6 (D+)
- net net_USB_VBUS: now also J_USB1.A4 (VBUS), J_USB1.A9 (VBUS), J_USB1.B4 (VBUS), J_USB1.B9 (VBUS)
- no-connect marks 46 -> 48
Changed lines of the file:
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@@
 	(generator "eeschema")
 	(generator_version "10.0")
-	(paper "A4")
+	(paper "User" 1300 400)
 	(title_block
 		(title "SWAFarm NODE_CORE")
@@
 )
 )
-(symbol (lib_id "Connector:USB_C_Receptacle_USB2.0_14P") (at 459.74 139.7 0) (unit 1)
+(symbol (lib_id "Connector:USB_C_Receptacle_16P") (at 459.74 139.7 0) (unit 1)
 (exclude_from_sim no) (in_bom yes) (on_board yes) (dnp no)
 	(property "Reference" "J_USB1" (at 459.74 134.61999999999998 0)
@@
 		(effects (font (size 1.27 1.27)) hide)
 	)
+	(pin "A8")
+	(pin "B8")
 	(pin "A1")
 	(pin "A4")
@@
 	(no_connect (at 415.29 137.16))
 	(no_connect (at 415.29 139.7))
+	(no_connect (at 474.98 147.32))
+	(no_connect (at 474.98 149.86))
 (symbol (lib_id "Device:R") (at 500.38 59.69 0) (unit 1)
 (exclude_from_sim no) (in_bom yes) (on_board yes) (dnp no)
@@
 	(no_connect (at 594.36 193.04))
 (symbol (lib_id "RF_Module:RAK3172-xx-8-SM-xI") (at 849.63 100.33 0) (unit 1)
-(exclude_from_sim no) (in_bom yes) (on_board yes) (dnp yes)
+(exclude_from_sim no) (in_bom yes) (on_board yes) (dnp no)
 	(property "Reference" "U_LORA1" (at 849.63 95.25 0)
 		(effects (font (size 1.27 1.27)))
@@
 )
 (symbol (lib_id "Device:R") (at 820.42 80.01 0) (unit 1)
-(exclude_from_sim no) (in_bom yes) (on_board yes) (dnp yes)
+(exclude_from_sim no) (in_bom yes) (on_board yes) (dnp no)
 	(property "Reference" "R_LORABOOT1" (at 820.42 74.93 0)
 		(effects (font (size 1.27 1.27)))
@@
 )
 (symbol (lib_id "Device:R") (at 820.42 95.25 0) (unit 1)
-(exclude_from_sim no) (in_bom yes) (on_board yes) (dnp yes)
+(exclude_from_sim no) (in_bom yes) (on_board yes) (dnp no)
 	(property "Reference" "R_LORARST1" (at 820.42 90.17 0)
 		(effects (font (size 1.27 1.27)))
@@
 )
 (symbol (lib_id "Connector:TestPoint") (at 805.18 80.01 0) (unit 1)
-(exclude_from_sim no) (in_bom yes) (on_board yes) (dnp yes)
+(exclude_from_sim no) (in_bom yes) (on_board yes) (dnp no)
 	(property "Reference" "TP_LORABOOT1" (at 805.18 74.93 0)
 		(effects (font (size 1.27 1.27)))
@@
 )
 (symbol (lib_id "Connector:TestPoint") (at 805.18 95.25 0) (unit 1)
-(exclude_from_sim no) (in_bom yes) (on_board yes) (dnp yes)
+(exclude_from_sim no) (in_bom yes) (on_board yes) (dnp no)
 	(property "Reference" "TP_LORARST1" (at 805.18 90.17 0)
 		(effects (font (size 1.27 1.27)))
@@
 )
 (symbol (lib_id "Connector:Conn_Coaxial") (at 849.63 59.69 0) (unit 1)
-(exclude_from_sim no) (in_bom yes) (on_board yes) (dnp yes)
+(exclude_from_sim no) (in_bom yes) (on_board yes) (dnp no)
 	(property "Reference" "J_LORASMA1" (at 849.63 54.61 0)
 		(effects (font (size 1.27 1.27)))
@@
 		(effects (font (size 1.27 1.27)))
 	)
-	(property "Footprint" "Package_SO:SOIC-8_3.9x4.9mm_P1.27mm" (at 1150.62 46.989999999999995 0)
+	(property "Footprint" "Package_SO:TI_SO-PowerPAD-8_ThermalVias" (at 1150.62 46.989999999999995 0)
 		(effects (font (size 1.27 1.27)) hide)
 	)
@@
 		(effects (font (size 1.27 1.27)))
 	)
-	(property "Footprint" "Package_SO:SOIC-8_3.9x4.9mm_P1.27mm" (at 1150.62 71.12 0)
+	(property "Footprint" "Package_SO:TI_SO-PowerPAD-8_ThermalVias" (at 1150.62 71.12 0)
 		(effects (font (size 1.27 1.27)) hide)
 	)
@@
 		(effects (font (size 1.27 1.27)))
 	)
-	(property "Footprint" "Package_SO:SOIC-8_3.9x4.9mm_P1.27mm" (at 1150.62 95.25 0)
+	(property "Footprint" "Package_SO:TI_SO-PowerPAD-8_ThermalVias" (at 1150.62 95.25 0)
 		(effects (font (size 1.27 1.27)) hide)
 	)
@@
 		(effects (font (size 1.27 1.27)))
 	)
-	(property "Footprint" "Package_SO:SOIC-8_3.9x4.9mm_P1.27mm" (at 1150.62 119.38000000000001 0)
+	(property "Footprint" "Package_SO:TI_SO-PowerPAD-8_ThermalVias" (at 1150.62 119.38000000000001 0)
 		(effects (font (size 1.27 1.27)) hide)
 	)
@@
 		(effects (font (size 1.27 1.27)))
 	)
-	(property "Footprint" "Package_SO:SOIC-8_3.9x4.9mm_P1.27mm" (at 1150.62 143.51 0)
+	(property "Footprint" "Package_SO:TI_SO-PowerPAD-8_ThermalVias" (at 1150.62 143.51 0)
 		(effects (font (size 1.27 1.27)) hide)
 	)
@@
 		(effects (font (size 1.27 1.27)))
 	)
-	(property "Footprint" "Package_SO:SOIC-8_3.9x4.9mm_P1.27mm" (at 1150.62 167.64000000000001 0)
+	(property "Footprint" "Package_SO:TI_SO-PowerPAD-8_ThermalVias" (at 1150.62 167.64000000000001 0)
 		(effects (font (size 1.27 1.27)) hide)
 	)

Commit message: updated
Parts:
- added F2: Polyfuse_4A, Fuse:Fuse_1812_4532Metric, symbol Device:Polyfuse
- added JP_IGND1, JP_IGND2, JP_IGND3, JP_IGND4, JP_IGND5, JP_IGND6: I_mode_gnd, Connector_PinHeader_2.54mm:PinHeader_1x02_P2.54mm_Vertical, symbol Connector_Generic:Conn_01x02
- added JP_VBYP1, JP_VBYP2, JP_VBYP3, JP_VBYP4, JP_VBYP5, JP_VBYP6: V_mode_bypass, Connector_PinHeader_2.54mm:PinHeader_1x02_P2.54mm_Vertical, symbol Connector_Generic:Conn_01x02
- added R_VBOT1, R_VBOT2, R_VBOT3, R_VBOT4, R_VBOT5, R_VBOT6: 100k, Resistor_SMD:R_0805_2012Metric, symbol Device:R
- added TP_VALVE_PWR1: V12_VALVE, TestPoint:TestPoint_Pad_D1.5mm, symbol Connector:TestPoint
- F1: value Polyfuse_1.5A -> Polyfuse_5A
- R_SER1, R_SER2, R_SER3, R_SER4, R_SER5, R_SER6: value 100k -> 232k
Connections:
- net GND: now also JP_IGND1.2 (Pin_2), JP_IGND2.2 (Pin_2), JP_IGND3.2 (Pin_2), JP_IGND4.2 (Pin_2), JP_IGND5.2 (Pin_2), JP_IGND6.2 (Pin_2), R_VBOT1.2, R_VBOT2.2, R_VBOT3.2, R_VBOT4.2, R_VBOT5.2, R_VBOT6.2; no longer R_BURDEN1.2, R_BURDEN2.2, R_BURDEN3.2, R_BURDEN4.2, R_BURDEN5.2, R_BURDEN6.2
- net SENSOR_CH1: now also JP_VBYP1.2 (Pin_2), R_VBOT1.1
- net SENSOR_CH2: now also JP_VBYP2.2 (Pin_2), R_VBOT2.1
- net SENSOR_CH3: now also JP_VBYP3.2 (Pin_2), R_VBOT3.1
- net SENSOR_CH4: now also JP_VBYP4.2 (Pin_2), R_VBOT4.1
- net SENSOR_CH5: now also JP_VBYP5.2 (Pin_2), R_VBOT5.1
- net SENSOR_CH6: now also JP_VBYP6.2 (Pin_2), R_VBOT6.1
- net V12_PROT: now also F2.1
- net V12_SW: no longer C_VALVEBULK1.1, C_VMDEC1.1, C_VMDEC2.1, C_VMDEC3.1, C_VMDEC4.1, C_VMDEC5.1, C_VMDEC6.1, U_DRV1.5 (VM), U_DRV2.5 (VM), U_DRV3.5 (VM), U_DRV4.5 (VM), U_DRV5.5 (VM), U_DRV6.5 (VM)
- net net_CH1_SIG: now also JP_VBYP1.1 (Pin_1)
- net net_CH2_SIG: now also JP_VBYP2.1 (Pin_1)
- net net_CH3_SIG: now also JP_VBYP3.1 (Pin_1)
- net net_CH4_SIG: now also JP_VBYP4.1 (Pin_1)
- net net_CH5_SIG: now also JP_VBYP5.1 (Pin_1)
- net net_CH6_SIG: now also JP_VBYP6.1 (Pin_1)
- new net V12_VALVE: C_VALVEBULK1.1, C_VMDEC1.1, C_VMDEC2.1, C_VMDEC3.1, C_VMDEC4.1, C_VMDEC5.1, C_VMDEC6.1, F2.2, TP_VALVE_PWR1.1, U_DRV1.5 (VM), U_DRV2.5 (VM), U_DRV3.5 (VM), U_DRV4.5 (VM), U_DRV5.5 (VM), U_DRV6.5 (VM)
- new net net_CH1_IGND: JP_IGND1.1 (Pin_1), R_BURDEN1.2
- new net net_CH2_IGND: JP_IGND2.1 (Pin_1), R_BURDEN2.2
- new net net_CH3_IGND: JP_IGND3.1 (Pin_1), R_BURDEN3.2
- new net net_CH4_IGND: JP_IGND4.1 (Pin_1), R_BURDEN4.2
- new net net_CH5_IGND: JP_IGND5.1 (Pin_1), R_BURDEN5.2
- new net net_CH6_IGND: JP_IGND6.1 (Pin_1), R_BURDEN6.2

Commit message: updated
Changed lines of the file:
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@@
 (symbol (lib_id "power:PWR_FLAG") (at 190.5 59.69 0) (unit 1)
 (exclude_from_sim no) (in_bom yes) (on_board yes) (dnp no)
-	(property "Reference" "FLAG6" (at 190.5 53.339999999999996 0)
+	(property "Reference" "#FLG06" (at 190.5 53.339999999999996 0)
 		(effects (font (size 1.27 1.27)))
 	)
@@
 (project "SWAFarmNodeV1"
 (path "/7f190bf9-c800-4055-b329-7f500a7a2cbd"
-(reference "FLAG6")
+(reference "#FLG06")
 (unit 1)
 )
