File: Hardware/SWAFarmNodeV1/SWAFarmNodeV1.kicad_sch (KiCad schematic)
At the start: 181 parts, among them J1 M12_5P_A_Coded_PowerIn, Q1 IPD50N06S4L-16, U1 TPS26600PWP, U2 TPS54561, U3 TPS563201

Commit message: Schematics Clean up phase-1 completed
Parts:
- removed C_VALVEBULK1: 1000uF_25V, Capacitor_THT:CP_Radial_D12.5mm_P5.00mm, symbol Device:C
- removed D_CLLO1, D_CLLO2, D_CLLO3, D_CLLO4, D_CLLO5, D_CLLO6: BAV99_2of2, Diode_SMD:D_SOD-123, symbol Device:D
- added C_VALVEBULK1, C_VALVEBULK2, C_VALVEBULK3, C_VALVEBULK4, C_VALVEBULK5, C_VALVEBULK6: 1000uF_25V, Capacitor_THT:CP_Radial_D12.5mm_P5.00mm, symbol Device:C_Polarized_US
- D_CLHI1, D_CLHI2, D_CLHI3, D_CLHI4, D_CLHI5, D_CLHI6: value BAV99_1of2 -> BAV99
- D_FLT1: value Red_FAULT -> Red
- D_LINK1: value Yellow_LINK -> Yellow
- D_PWR1: value Green_PWR -> Green
- J1: value M12_5P_A_Coded_PowerIn -> PWR JACK
- J_OUT1: value M12_5P_A_Coded_PowerOut -> M12_5P
- R_BURDEN1, R_BURDEN2, R_BURDEN3, R_BURDEN4, R_BURDEN5, R_BURDEN6: value 150_0.1pct -> 150R
- R_ILIM_V1, R_ILIM_V2, R_ILIM_V3, R_ILIM_V4, R_ILIM_V5, R_ILIM_V6: value 20k_TBD -> 20k
- R_TERM1: value 120_SOLDER_SELECT -> 120R
Connections:
- net GND: now also D_CLHI1.1 (K), D_CLHI2.1 (K), D_CLHI3.1 (K), D_CLHI4.1 (K), D_CLHI5.1 (K), D_CLHI6.1 (K), C_VALVEBULK1.2, C_VALVEBULK2.2, C_VALVEBULK3.2, C_VALVEBULK4.2, C_VALVEBULK5.2, C_VALVEBULK6.2
- net SENSOR_CH1: now also D_CLHI1.3 (A/K); no longer D_CLHI1.2 (A)
- net SENSOR_CH2: now also D_CLHI2.3 (A/K); no longer D_CLHI2.2 (A)
- net SENSOR_CH3: now also D_CLHI3.3 (A/K); no longer D_CLHI3.2 (A)
- net SENSOR_CH4: now also D_CLHI4.3 (A/K); no longer D_CLHI4.2 (A)
- net SENSOR_CH5: now also D_CLHI5.3 (A/K); no longer D_CLHI5.2 (A)
- net SENSOR_CH6: now also D_CLHI6.3 (A/K); no longer D_CLHI6.2 (A)
- net V12_VALVE: now also C_VALVEBULK1.1, C_VALVEBULK2.1, C_VALVEBULK3.1, C_VALVEBULK4.1, C_VALVEBULK5.1, C_VALVEBULK6.1
- net V3V3_RAIL: no longer C_BULK2.1, C_DEC1.1, C_DEC10.1, C_DEC2.1, C_DEC3.1, C_DEC4.1, C_DEC5.1, C_DEC6.1, C_DEC7.1, C_DEC8.1, C_DEC9.1, D_CLHI1.1 (K), D_CLHI2.1 (K), D_CLHI3.1 (K), D_CLHI4.1 (K), D_CLHI5.1 (K), D_CLHI6.1 (K), R_BOOT1.1, R_ENPU1.1, R_EXPRST1.1, R_LORARST1.1, R_SETUP1.1, U_ISO1.1 (Vcc1), U_LORA1.24 (VDD), U_MCU1.2 (3V3), U_VALVEEXP1.9 (V_{DD})
- net V5_RAIL: no longer C_ISOIN1.1, U_ISODCDC1.2 (+Vin)
- net net_CH1_IGND: no longer names the net of JP_IGND1.1 (Pin_1), R_BURDEN1.2
- net net_CH2_IGND: no longer names the net of JP_IGND2.1 (Pin_1), R_BURDEN2.2
- net net_CH3_IGND: no longer names the net of JP_IGND3.1 (Pin_1), R_BURDEN3.2
- net net_CH4_IGND: no longer names the net of JP_IGND4.1 (Pin_1), R_BURDEN4.2
- net net_CH5_IGND: no longer names the net of JP_IGND5.1 (Pin_1), R_BURDEN5.2
- net net_CH6_IGND: no longer names the net of JP_IGND6.1 (Pin_1), R_BURDEN6.2
- net net_ISO_5V renamed ISO_5V
- net net_ISO_GND renamed ISO_GND
- net net_LEDFLT_A: no longer names the net of D_FLT1.2 (A), R_LEDFLT1.2
- net net_LEDLINK_A: no longer names the net of D_LINK1.2 (A), R_LINK1.2
- net net_LEDPWR_A: no longer names the net of D_PWR1.2 (A), R_PWR1.2
- net net_LORA_RF renamed LORA_RF
- net net_V1_ILIM: no longer names the net of R_ILIM_V1.1, U_DRV1.4 (ILIM)
- net net_V2_ILIM: no longer names the net of R_ILIM_V2.1, U_DRV2.4 (ILIM)
- net net_V3_ILIM: no longer names the net of R_ILIM_V3.1, U_DRV3.4 (ILIM)
- net net_V4_ILIM: no longer names the net of R_ILIM_V4.1, U_DRV4.4 (ILIM)
- net net_V5_ILIM: no longer names the net of R_ILIM_V5.1, U_DRV5.4 (ILIM)
- net net_V6_ILIM: no longer names the net of R_ILIM_V6.1, U_DRV6.4 (ILIM)
- new net +3V3: C_BULK2.1, C_DEC1.1, C_DEC10.1, C_DEC2.1, C_DEC3.1, C_DEC4.1, C_DEC5.1, C_DEC6.1, C_DEC7.1, C_DEC8.1, C_DEC9.1, D_CLHI1.2 (A), D_CLHI2.2 (A), D_CLHI3.2 (A), D_CLHI4.2 (A), D_CLHI5.2 (A), D_CLHI6.2 (A), R_BOOT1.1, R_ENPU1.1, R_EXPRST1.1, R_LORARST1.1, R_SETUP1.1, U_ISO1.1 (Vcc1), U_LORA1.24 (VDD), U_MCU1.2 (3V3), U_VALVEEXP1.9 (V_{DD})
- new net +5V: C_ISOIN1.1, U_ISODCDC1.2 (+Vin)
Other:
- moved on the sheet: CMC_RS485_1, CMC_RS485_2, C_BOOT1, C_BOOT2, C_BULK2, C_COMP1, C_DEC1, C_DEC10, C_DEC2, C_DEC3, C_DEC4, C_DEC5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

Commit message: Schematics Clean up Phase-2 Completed
Connections:
- net +3V3: now also C_OUT3.1, D_LED2.1 (K), L2.2, R_FB2A1.1
- net +5V: now also C_IN3.1, C_OUT2.1, L1.2, R_EN2.1, R_FB1A1.1, R_LED1.2, R_PG1.1, TP_5V1.1, U3.3 (VIN)
- net V12_PROT renamed VIN_12V
- net V12_SW renamed 12V_SW
- net 12V_SW: now also R_FLT1.2
- net V12_VALVE renamed +12V
- removed net V3V3_RAIL: C_OUT3.1, D_LED2.1 (K), L2.2, R_FB2A1.1, TP_3V3.1
- removed net V5_RAIL: C_IN3.1, C_OUT2.1, L1.2, R_EN2.1, R_FB1A1.1, R_FLT1.2, R_LED1.2, R_PG1.1, TP_5V1.1, U3.3 (VIN)
- net net_BOOT1: no longer names the net of C_BOOT1.1, U2.1 (BOOT)
- net net_BOOT2: no longer names the net of C_BOOT2.1, U3.6 (VBST)
- net net_COMP1: no longer names the net of R_COMP1.1, U2.7 (COMP)
- net net_COMPA: no longer names the net of C_COMP1.1, R_COMP1.2
- net net_DVDT: no longer names the net of C_DVDT1.1, U1.12 (dVdT)
- net net_EN1: no longer names the net of R_EN1A1.2, R_EN1B1.1, U2.3 (EN)
- net net_EN2: no longer names the net of R_EN2.2, U3.5 (EN)
- net net_FB1MID: no longer names the net of R_FB1A1.2, R_FB1B1.1, U2.6 (FB)
- net net_FB2MID: no longer names the net of R_FB2A1.2, R_FB2B1.1, U3.4 (VFB)
- net net_FLT: no longer names the net of R_FLT1.1, TP_FLT1.1, U1.14 (~{FLT})
- net net_ILIM: no longer names the net of R_ILIM1.1, U1.11 (ILIM)
- net net_IMON: no longer names the net of R_IMON1.1, TP_IMON1.1, U1.10 (IMON)
- net net_LED1A: no longer names the net of D_LED1.2 (A), R_LED1.1
- net net_LED2A: no longer names the net of D_LED2.2 (A), R_LED2.1
- net net_OVP: no longer names the net of R_OVP1.2, R_OVP2.1, U1.5 (OVP)
- net net_PWRGD: no longer names the net of D_LED1.1 (K), R_PG1.2, TP_PG1.1, U2.10 (PWRGD)
- net net_RT1: no longer names the net of R_RT1.1, U2.5 (RT/CLK)
- net net_SHDN: no longer names the net of R_SHDN1.2, U1.7 (~{SHDN})
- net net_SS1: no longer names the net of C_SS1.1, U2.4 (SS/TR)
- net net_SW1: no longer names the net of C_BOOT1.2, L1.1, U2.9 (SW)
- net net_SW2: no longer names the net of C_BOOT2.2, L2.1, U3.2 (SW)
- net net_UVLO: no longer names the net of R_UVLO1.2, R_UVLO2.1, U1.3 (UVLO)
Other:
- moved on the sheet: C_BOOT1, C_BOOT2, C_COMP1, C_DVDT1, C_IN3, C_OUT2, C_OUT3, C_SS1, D_LED1, D_LED2, F2, J_OUT1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

Commit message: Schematics Cleanup Done
Parts:
- removed CMC_RS485_1, CMC_RS485_2: 744232090, Inductor_SMD:L_CommonModeChoke_Bourns_SRF1260, symbol Device:Filter_EMI_CommonMode
- removed C_BOOT1, C_BOOT2, C_DEC1, C_DEC10, C_DEC2, C_DEC3, C_DEC4, C_DEC5, C_DEC6, C_DEC7, C_DEC8, C_DEC9, C_FILT1, C_FILT2, C_FILT3, C_FILT4, C_FILT5, C_FILT6, C_ISOIN1, C_ISOOUT1: 100nF, Capacitor_SMD:C_0603_1608Metric, symbol Device:C
- removed C_BULK2: 10uF, Capacitor_SMD:C_1206_3216Metric, symbol Device:C
- removed C_COMP1: 2.2nF_TBD, Capacitor_SMD:C_0603_1608Metric, symbol Device:C
- removed C_DVDT1: 1nF_TBD, Capacitor_SMD:C_0805_2012Metric, symbol Device:C
- removed C_EN1, C_VMDEC1, C_VMDEC2, C_VMDEC3, C_VMDEC4, C_VMDEC5, C_VMDEC6: 1uF, Capacitor_SMD:C_0805_2012Metric, symbol Device:C
- removed C_IN1, C_IN2, C_OUT1: 10uF_25V, Capacitor_SMD:C_1206_3216Metric, symbol Device:C
- removed C_IN3: 10uF_16V, Capacitor_SMD:C_1206_3216Metric, symbol Device:C
- removed C_OUT2, C_OUT3: 22uF_10V, Capacitor_SMD:C_1206_3216Metric, symbol Device:C
- removed C_SS1: 10nF_TBD, Capacitor_SMD:C_0603_1608Metric, symbol Device:C
- removed C_VALVEBULK1, C_VALVEBULK2, C_VALVEBULK3, C_VALVEBULK4, C_VALVEBULK5, C_VALVEBULK6: 1000uF_25V, Capacitor_THT:CP_Radial_D12.5mm_P5.00mm, symbol Device:C_Polarized_US
- removed D1: SMBJ18CA, Diode_SMD:D_SMB, symbol Device:D_TVS_Filled
- removed D_CLHI1, D_CLHI2, D_CLHI3, D_CLHI4, D_CLHI5, D_CLHI6: BAV99, Diode_SMD:D_SOD-123, symbol Device:D
- removed D_FLT1: Red, LED_SMD:LED_0805_2012Metric, symbol Device:LED
- removed D_LED1: Green_PowerGood, LED_SMD:LED_0805_2012Metric, symbol Device:LED
- removed D_LED2: Green_3V3Present, LED_SMD:LED_0805_2012Metric, symbol Device:LED
- removed D_LINK1: Yellow, LED_SMD:LED_0805_2012Metric, symbol Device:LED
- removed D_PWR1: Green, LED_SMD:LED_0805_2012Metric, symbol Device:LED
- removed D_RS485PROT1, D_RS485PROT2: SM712-02HTG, Package_TO_SOT_SMD:SOT-23, symbol Diode:SM712_SOT23
- removed F1: Polyfuse_5A, Fuse:Fuse_1812_4532Metric, symbol Device:Polyfuse
- removed F2: Polyfuse_4A, Fuse:Fuse_1812_4532Metric, symbol Device:Polyfuse
- removed J1: PWR JACK, Connector_PinHeader_2.54mm:PinHeader_1x04_P2.54mm_Vertical, symbol Connector_Generic:Conn_01x04
- removed JP_IGND1, JP_IGND2, JP_IGND3, JP_IGND4, JP_IGND5, JP_IGND6: I_mode_gnd, Connector_PinHeader_2.54mm:PinHeader_1x02_P2.54mm_Vertical, symbol Connector_Generic:Conn_01x02
- removed JP_VBYP1, JP_VBYP2, JP_VBYP3, JP_VBYP4, JP_VBYP5, JP_VBYP6: V_mode_bypass, Connector_PinHeader_2.54mm:PinHeader_1x02_P2.54mm_Vertical, symbol Connector_Generic:Conn_01x02
- removed J_LORASMA1: SMA_Bulkhead_Antenna, Connector_Coaxial:SMA_Amphenol_132134_Vertical, symbol Connector:Conn_Coaxial
- removed J_OUT1: M12_5P, Connector_PinHeader_2.54mm:PinHeader_1x04_P2.54mm_Vertical, symbol Connector_Generic:Conn_01x04
- removed J_PROG1: Debug_UART_TX_RX_GND, Connector_PinHeader_2.54mm:PinHeader_1x03_P2.54mm_Vertical, symbol Connector_Generic:Conn_01x03
- removed J_RS485_IN1: M12_5P_A_Coded_RS485_Bus_In, Connector_PinHeader_2.54mm:PinHeader_1x05_P2.54mm_Vertical, symbol Connector_Generic:Conn_01x05
- removed J_RS485_LOC1: M12_5P_A_Coded_RS485_Local, Connector_PinHeader_2.54mm:PinHeader_1x05_P2.54mm_Vertical, symbol Connector_Generic:Conn_01x05
- removed J_RS485_OUT1: M12_5P_A_Coded_RS485_Bus_Out, Connector_PinHeader_2.54mm:PinHeader_1x05_P2.54mm_Vertical, symbol Connector_Generic:Conn_01x05
- removed J_SENSOR_RET1: SensorReturn_x6, TerminalBlock_Phoenix:TerminalBlock_Phoenix_MKDS-1,5-6-5.08_1x06_P5.08mm_Horizontal, symbol Connector_Generic:Conn_01x06
- removed J_SENSOR_SIG1: SensorSignal_x6, TerminalBlock_Phoenix:TerminalBlock_Phoenix_MKDS-1,5-6-5.08_1x06_P5.08mm_Horizontal, symbol Connector_Generic:Conn_01x06
- removed J_USB1: USB-C_Programming, Connector_USB:USB_C_Receptacle_HRO_TYPE-C-31-M-12, symbol Connector:USB_C_Receptacle_16P
- removed J_VALVE_OUT1_1: ValveOut1_x6, TerminalBlock_Phoenix:TerminalBlock_Phoenix_MKDS-1,5-6-5.08_1x06_P5.08mm_Horizontal, symbol Connector_Generic:Conn_01x06
- removed J_VALVE_OUT2_1: ValveOut2_x6, TerminalBlock_Phoenix:TerminalBlock_Phoenix_MKDS-1,5-6-5.08_1x06_P5.08mm_Horizontal, symbol Connector_Generic:Conn_01x06
- removed L1: 3.3uH_TBD, Inductor_SMD:L_Bourns-SRN6028, symbol Device:L
- removed L2: 2.2uH_TBD, Inductor_SMD:L_Bourns-SRN4018, symbol Device:L
- removed Q1: IPD50N06S4L-16, Package_TO_SOT_SMD:SOT-23, symbol Transistor_FET:Q_NMOS_GSD
- removed R_BIASA1, R_BIASB1: 680, Resistor_SMD:R_0805_2012Metric, symbol Device:R
- removed R_BOOT1, R_EN1B1, R_ENPU1, R_EXPRST1, R_FB1B1, R_FB2B1, R_FLT1, R_IMON1, R_LORABOOT1, R_LORARST1, R_OVP2, R_PG1, R_SETUP1, R_UVLO2, R_gate1: 10k, Resistor_SMD:R_0805_2012Metric, symbol Device:R
- removed R_BURDEN1, R_BURDEN2, R_BURDEN3, R_BURDEN4, R_BURDEN5, R_BURDEN6: 150R, Resistor_SMD:R_0805_2012Metric, symbol Device:R
- removed R_CC1_1, R_CC2_1: 5.1k, Resistor_SMD:R_0805_2012Metric, symbol Device:R
- removed R_COMP1: 10k_TBD, Resistor_SMD:R_0805_2012Metric, symbol Device:R
- removed R_EN1A1: 73.2k_TBD, Resistor_SMD:R_0805_2012Metric, symbol Device:R
- removed R_EN2, R_SHDN1, R_VBOT1, R_VBOT2, R_VBOT3, R_VBOT4, R_VBOT5, R_VBOT6: 100k, Resistor_SMD:R_0805_2012Metric, symbol Device:R
- removed R_FB1A1: 52.3k, Resistor_SMD:R_0805_2012Metric, symbol Device:R
- removed R_FB2A1: 32.4k, Resistor_SMD:R_0805_2012Metric, symbol Device:R
- removed R_ILIM1: 20k_TBD, Resistor_SMD:R_0805_2012Metric, symbol Device:R
- removed R_ILIM_V1, R_ILIM_V2, R_ILIM_V3, R_ILIM_V4, R_ILIM_V5, R_ILIM_V6: 20k, Resistor_SMD:R_0805_2012Metric, symbol Device:R
- removed R_LED1, R_LEDFLT1, R_LINK1, R_PWR1: 1k, Resistor_SMD:R_0805_2012Metric, symbol Device:R
- removed R_LED2: 330, Resistor_SMD:R_0805_2012Metric, symbol Device:R
- removed R_OVP1: 124k, Resistor_SMD:R_0805_2012Metric, symbol Device:R
- removed R_RT1: 100k_TBD, Resistor_SMD:R_0805_2012Metric, symbol Device:R
- removed R_SER1, R_SER2, R_SER3, R_SER4, R_SER5, R_SER6: 232k, Resistor_SMD:R_0805_2012Metric, symbol Device:R
- removed R_TERM1: 120R, Resistor_SMD:R_0805_2012Metric, symbol Device:R
- removed R_UVLO1: 64.9k, Resistor_SMD:R_0805_2012Metric, symbol Device:R
- removed SW_BOOT1: BOOT, Button_Switch_SMD:SW_SPST_B3U-1000P, symbol Switch:SW_Push
- removed SW_RESET1: RESET, Button_Switch_SMD:SW_SPST_B3U-1000P, symbol Switch:SW_Push
- removed SW_SETUP1: SETUP, Button_Switch_SMD:SW_SPST_B3U-1000P, symbol Switch:SW_Push
- removed TP_12V_SW1: V12_SW, TestPoint:TestPoint_Pad_D1.5mm, symbol Connector:TestPoint
- removed TP_3V3: V3V3_RAIL, TestPoint:TestPoint_Pad_D1.5mm, symbol Connector:TestPoint
- removed TP_5V1: V5_RAIL, TestPoint:TestPoint_Pad_D1.5mm, symbol Connector:TestPoint
- removed TP_FLT1: nFLT, TestPoint:TestPoint_Pad_D1.5mm, symbol Connector:TestPoint
- removed TP_GND1: GND, TestPoint:TestPoint_Pad_D1.5mm, symbol Connector:TestPoint
- removed TP_IMON1: IMON, TestPoint:TestPoint_Pad_D1.5mm, symbol Connector:TestPoint
- removed TP_ISO5V1: ISO_5V, TestPoint:TestPoint_Pad_D1.5mm, symbol Connector:TestPoint
- removed TP_ISOGND1: ISO_GND, TestPoint:TestPoint_Pad_D1.5mm, symbol Connector:TestPoint
- removed TP_LORABOOT1: LORA_BOOT0, TestPoint:TestPoint_Pad_D1.5mm, symbol Connector:TestPoint
- removed TP_LORARST1: LORA_RESET, TestPoint:TestPoint_Pad_D1.5mm, symbol Connector:TestPoint
- removed TP_PG1: nPWRGD, TestPoint:TestPoint_Pad_D1.5mm, symbol Connector:TestPoint
- removed TP_RS485DI1: ISO_DI, TestPoint:TestPoint_Pad_D1.5mm, symbol Connector:TestPoint
- removed TP_RS485RO1: ISO_RO, TestPoint:TestPoint_Pad_D1.5mm, symbol Connector:TestPoint
- removed TP_USBVBUS1: USB_VBUS, TestPoint:TestPoint_Pad_D1.5mm, symbol Connector:TestPoint
- removed TP_VALVE_PWR1: V12_VALVE, TestPoint:TestPoint_Pad_D1.5mm, symbol Connector:TestPoint
- removed U1: TPS26600PWP, Package_SO:HTSSOP-16-1EP_4.4x5mm_P0.65mm_EP3.4x5mm_Mask2.66x2.46mm_ThermalVias, symbol Power_Management:TPS26600PWP
- removed U2: TPS54561, Package_SON:WSON-10-1EP_4x4mm_P0.8mm_EP2.6x3mm_ThermalVias, symbol Regulator_Switching:TPS54561
- removed U3: TPS563201, Package_TO_SOT_SMD:SOT-23-6, symbol Regulator_Switching:TPS563201
- removed U_DRV1, U_DRV2, U_DRV3, U_DRV4, U_DRV5, U_DRV6: DRV8871DDAR, Package_SO:TI_SO-PowerPAD-8_ThermalVias, symbol Driver_Motor:DRV8871DDA
- removed U_ISO1: ISO7761DW, Package_SO:SOIC-16W_7.5x10.3mm_P1.27mm, symbol Isolator:ISO7761DW
- removed U_ISODCDC1: MEE1S0505SC, Converter_DCDC:Converter_DCDC_Murata_MEE1SxxxxSC_THT, symbol Converter_DCDC_Isolated:MEE1S0505SC
- removed U_LORA1: RAK3172-xx-8-SM-xI, RF_Module:RAK3172, symbol RF_Module:RAK3172-xx-8-SM-xI
- removed U_MCU1: ESP32-S3-WROOM-1-N16R8, RF_Module:ESP32-S3-WROOM-1, symbol RF_Module:ESP32-S3-WROOM-1
- removed U_RS485_TX1: THVD1450DR, Package_SO:SOIC-8_3.9x4.9mm_P1.27mm, symbol Interface_UART:THVD1450DR
- removed U_VALVEEXP1: MCP23S17-E/SO, Package_SO:SOIC-28W_7.5x17.9mm_P1.27mm, symbol Interface_Expansion:MCP23S17x-x-SO
Connections:
- no-connect marks 48 -> 0
Other:
- added sheet MCU (MCU.kicad_sch)
- added sheet Motor Valve (Motor Valve.kicad_sch)
- added sheet Power (Power.kicad_sch)
- added sheet RS-485 (RS-485.kicad_sch)
- added sheet Sensors & LORA (Sensors & LORA.kicad_sch)
