File: Hardware/SWAFarmNodeV1_STM32_ARCHIVE/SWAFarmNodeV1.kicad_pcb (KiCad board)
At the start: 4 copper layers, 300 x 220 mm, 203 parts, among them J1 DC_IN_12V, J2 SOLAR_IN_12V_class, J3 4S_LiFePO4_Pack, Q1 NMOS_30V_RDSon_20mOhm, Q2 NMOS_30V_RDSon_20mOhm, U1 LT8610AC-3.3

Commit message: uodated with Murli BOM
Parts:
- moved FB_MCU1 39.4 mm to (150.0, 132.0)
- moved C_SYS1 32.4 mm to (63.0, 78.0)
- moved C_MCU_BULK1 26.5 mm to (162.0, 126.0)
- moved C_MCU_VDD3 26.5 mm to (138.0, 126.0)
- moved C_MCU_VDD2 20.0 mm to (138.0, 120.0)
- moved C_MCU_VDDUSB1 20.0 mm to (162.0, 120.0)
- moved C_MCU_VDD1 15.7 mm to (138.0, 114.0)
- moved C_MCU_VDDA2 15.7 mm to (162.0, 114.0)
- moved C_MCU_VBAT1 15.3 mm to (138.0, 108.0)
- moved C_MCU_VDDA1 15.3 mm to (162.0, 108.0)
- moved C_REGN1 13.0 mm to (63.0, 71.0)
- moved C_PMID1 12.6 mm to (63.0, 64.0)
